File: Atrium PCB/Atrium PCB.kicad_sch (KiCad schematic)
At the start: 167 parts, among them J1 Conn_01x05_Pin, SW1 EC11E09244BS, SW10 SW_Push, SW11 SW_Push, SW12 SW_Push, SW13 SW_Push, SW14 SW_Push, SW15 SW_Push, SW16 SW_Push, SW17 SW_Push, SW18 SW_Push, SW19 SW_Push, SW2 SKRPACE010, SW20 SW_Push, SW21 SW_Push, SW22 SW_Push, SW23 SW_Push, SW24 SW_Push, SW25 SW_Push, SW26 SW_Push, SW27 SW_Push, SW28 SW_Push, SW29 SW_Push, SW3 SKRPACE010, SW30 SW_Push, SW31 SW_Push, SW32 SW_Push, SW33 SW_Push, SW34 SW_Push, SW35 SW_Push, SW36 SW_Push, SW37 SW_Push, SW38 SW_Push, SW39 SW_Push, SW4 SW_Push, SW40 SW_Push, SW41 SW_Push, SW42 SW_Push, SW43 SW_Push, SW44 SW_Push, SW45 SW_Push, SW46 SW_Push, SW47 SW_Push, SW48 SW_Push, SW49 SW_Push, SW5 SW_Push, SW6 SW_Push, SW7 SW_Push, SW8 SW_Push, SW9 SW_Push, U12 AP2112K-3.3, U4 SN74LVC1T45DBVR, X1 X322512MSB4SI

Commit message: sync
Parts:
- removed C44, C46, C47, C48: 100nF, Capacitor_SMD:C_0603_1608Metric, symbol Device:C
- removed C45: 10uF, Capacitor_SMD:C_0805_2012Metric, symbol Device:C
- removed D10, D15, D19, D23, D27, D31, D35, D39, D4: D, symbol Device:D
- removed LED10, LED7, LED8, LED9: SK6812MINI-E_C5149201, easyeda2kicad:LED-SMD_4P-L3.2-W2.8-LS5.9_SK6812MINI-E, symbol easyeda2kicad:SK6812MINI-E_C5149201
- removed R19, R9: 470, Resistor_SMD:R_0603_1608Metric, symbol Device:R
- removed SW12, SW17, SW21, SW25, SW29, SW33, SW37, SW41, SW7: SW_Push, symbol Switch:SW_Push
- removed U4: SN74LVC1T45DBVR, easyeda2kicad:SOT-23-6_L2.9-W1.6-P0.95-LS2.8-BR, symbol easyeda2kicad:SN74LVC1T45DBVR
- added C100, C101, C102, C103, C104, C105, C106, C107, C108, C109, C110, C111, C112, C113, C114, C115, C116, C117, C118, C119, C120, C121, C122, C123, C124, C125, C126, C127, C128, C129, C130, C131, C132, C133, C134, C135, C136, C137, C138, C139, C140, C141, C142, C143, C144, C145, C146, C147, C148, C149, C150, C151, C152, C153, C154, C155, C156, C157, C158, C159, C160, C161, C162, C163, C164, C165, C166, C167, C168, C169, C170, C171, C172, C173, C174, C175, C176, C177, C178, C179, C180, C181, C182, C183, C184, C185, C186, C187, C188, C189, C190, C191, C192, C193, C194, C195, C196, C197, C198, C199, C200, C201, C202, C203, C204, C205, C206, C207, C208, C209, C210, C217, C218, C219, C220, C221, C222, C223, C224, C225, C226, C49, C50, C51, C52, C53, C54, C55, C56, C57, C58, C59, C60, C61, C68, C69, C70, C71, C72, C73, C74, C75, C76, C77, C78, C79, C80, C81, C82, C83, C84, C85, C86, C87, C88, C89, C90, C91, C92, C93, C94, C95, C96, C97, C98, C99: 100nF, Capacitor_SMD:C_0603_1608Metric, symbol Device:C
- added C211, C212, C213, C214, C215, C216: 22uF, Capacitor_SMD:C_0402_1005Metric, symbol Device:C
- added C301, C382, C383, C384, C385, C386, C387: 100nF, Capacitor_SMD:C_0402_1005Metric, symbol Device:C
- added D48, D49, D50, D51, D52: D, symbol Device:D
- added LED175, LED176, LED177, LED178, LED179, LED180, LED181, LED182, LED183, LED184, LED185, LED186, LED187, LED188, LED189, LED190, LED191, LED192, LED193, LED194, LED195, LED196, LED197, LED198, LED199, LED200, LED201, LED202, LED203, LED204, LED205, LED206, LED207, LED208, LED209, LED210, LED211, LED212, LED213, LED214, LED215, LED216, LED217, LED218, LED219, LED220, LED221, LED222, LED223, LED224, LED225, LED226, LED227, LED228, LED229, LED230, LED231, LED232, LED233, LED234, LED235, LED236, LED237, LED238, LED239, LED240, LED241, LED242, LED243, LED244, LED245, LED246, LED247, LED248, LED249, LED250, LED251, LED252, LED253, LED254, LED255, LED256, LED257, LED258, LED259, LED260, LED261, LED262, LED263, LED264, LED265, LED266, LED267, LED268, LED269, LED270, LED271, LED272, LED273, LED274, LED275, LED276, LED277, LED278, LED279, LED280, LED281, LED282, LED283, LED284, LED285, LED286, LED287, LED288, LED289, LED290, LED291, LED292, LED293, LED294, LED295, LED296, LED297, LED298, LED299, LED300, LED301, LED302, LED303, LED304, LED305, LED306, LED307, LED308, LED309, LED310, LED311, LED312, LED313, LED314, LED315, LED316, LED317, LED318, LED319, LED320, LED321, LED322, LED323, LED324, LED325, LED326, LED327, LED328, LED329, LED330, LED331, LED332, LED333, LED334, LED335, LED336, LED337, LED338, LED339, LED340, LED341, LED342: SK6812MINI-E_C5149201, easyeda2kicad:LED-SMD_4P-L3.2-W2.8-LS5.9_SK6812MINI-E, symbol easyeda2kicad:SK6812MINI-E_C5149201
- added R11, R12, R13, R14, R15, R16: 470, Resistor_SMD:R_0603_1608Metric, symbol Device:R
- added SW50, SW51, SW52, SW53, SW54: SW_Push, symbol Switch:SW_Push
- added U1: SN74LVC8T245, symbol Logic_LevelTranslator:SN74LVC8T245
Connections:
- net +5V is gone; now on net GND: C67.2
- net +3.3V: now also U1.1 (V_{CCA}), U1.2 (DIR); no longer C66.2
- net COL_1: now also R11.2, R12.2, R13.2, R14.2, R15.2, R16.2, U1.21 (B1)
- net COL_10: no longer SW45.1
- net COL_2: now also U1.20 (B2)
- net COL_3: now also U1.19 (B3); no longer SW46.1
- net COL_4: now also SW46.1, U1.18 (B4); no longer SW13.1
- net COL_5: now also SW13.1, U1.17 (B5); no longer SW8.1
- net COL_6: now also SW8.1, U1.16 (B6); no longer SW47.1
- net COL_7: now also SW47.1; no longer SW48.1
- net COL_8: now also SW48.1; no longer SW49.1
- net COL_9: now also SW49.1
- net GND: now also C66.2, C100.2, C101.2, C102.2, C103.2, C104.2, C105.2, C106.2, C107.2, C108.2, C109.2, C110.2, C111.2, C112.2, C113.2, C114.2, C115.2, C116.2, C117.2, C118.2, C119.2, C120.2, C121.2, C122.2, C123.2, C124.2, C125.2, C126.2, C127.2, C128.2, C129.2, C130.2, C131.2, C132.2, C133.2, C134.2, C135.2, C136.2, C137.2, C138.2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; no longer C66.1, C67.1
- net ROW_1: now also D43.1 (K), RP2350.16 (GPIO12), D50.1 (K); no longer RP2350.14 (GPIO10)
- net ROW_2: now also RP2350.17 (GPIO13), D48.1 (K), D51.1 (K); no longer RP2350.15 (GPIO11)
- net ROW_3: now also RP2350.18 (GPIO14), D49.1 (K), D52.1 (K); no longer RP2350.16 (GPIO12)
- net ROW_4: now also D11.1 (K), D44.1 (K), D45.1 (K), D46.1 (K), D47.1 (K), D6.1 (K), RP2350.19 (GPIO15); no longer D43.1 (K), RP2350.17 (GPIO13)
- net 5V_A1: now reaches RP2350.27 (GPIO16)
- net 5V_A1: now also U1.3 (A1)
- net 5V_A2: now reaches RP2350.28 (GPIO17)
- net 5V_A2: now also U1.4 (A2)
- net 5V_A3: now reaches RP2350.29 (GPIO18)
- net 5V_A3: now also U1.5 (A3)
- removed net ROW_5: D11.1 (K), D44.1 (K), D45.1 (K), D46.1 (K), D47.1 (K), D6.1 (K), RP2350.18 (GPIO14)
- net RP2350_GPIO_19 renamed 5V_A4
- net 5V_A4: now also U1.6 (A4)
- net RP2350_GPIO_20 renamed 5V_A5
- net 5V_A5: now also U1.7 (A5)
- net RP2350_GPIO_21 renamed 5V_A6
- net 5V_A6: now also U1.8 (A6)
- new net: LED321.2 (DIN), LED328.4 (DOUT)
- new net: LED315.2 (DIN), LED321.4 (DOUT)
- new net: D48.2 (A), SW50.2
- new net: LED302.2 (DIN), LED309.4 (DOUT)
- new net: LED295.2 (DIN), LED302.4 (DOUT)
- new net: LED241.2 (DIN), LED248.4 (DOUT)
- new net: LED234.2 (DIN), LED241.4 (DOUT)
- new net: D49.2 (A), SW51.2
- new net: LED207.4 (DOUT), LED214.2 (DIN)
- new net: LED214.4 (DOUT), LED221.2 (DIN)
- new net: C216.1, C387.2
- new net: LED264.2 (DIN), R14.1
- new net: LED264.4 (DOUT), LED271.2 (DIN)
- new net: LED245.4 (DOUT), LED252.2 (DIN)
- new net: LED252.4 (DOUT), LED253.2 (DIN)
- new net: LED319.4 (DOUT), LED326.2 (DIN)
- new net: LED326.4 (DOUT), LED333.2 (DIN)
- new net: LED305.4 (DOUT), LED312.2 (DIN)
- new net: LED308.4 (DOUT), LED309.2 (DIN)
- new net: LED307.2 (DIN), LED314.4 (DOUT)
- new net: LED300.2 (DIN), LED307.4 (DOUT)
- new net: LED234.4 (DOUT), LED235.2 (DIN)
- new net: LED233.4 (DOUT), LED240.2 (DIN)
- new net: LED240.4 (DOUT), LED247.2 (DIN)
- new net: LED271.4 (DOUT), LED278.2 (DIN)
- new net: LED278.4 (DOUT), LED285.2 (DIN)
- new net: LED285.4 (DOUT), LED286.2 (DIN)
- new net: LED279.2 (DIN), LED286.4 (DOUT)
- new net: LED280.4 (DOUT), LED281.2 (DIN)
- new net: LED274.2 (DIN), LED281.4 (DOUT)
- new net: LED246.2 (DIN), LED253.4 (DOUT)
- new net: LED197.2 (DIN), LED198.4 (DOUT)
- new net: LED196.2 (DIN), LED197.4 (DOUT)
- new net: LED208.2 (DIN), R12.1
- new net: LED206.2 (DIN), LED213.4 (DOUT)
- new net: LED206.4 (DOUT), LED207.2 (DIN)
- new net: LED179.4 (DOUT), LED180.2 (DIN)
- new net: LED180.4 (DOUT), LED181.2 (DIN)
- new net: LED226.4 (DOUT), LED227.2 (DIN)
- new net: LED220.2 (DIN), LED227.4 (DOUT)
- new net: LED188.2 (DIN), LED189.4 (DOUT)
- new net: LED187.2 (DIN), LED188.4 (DOUT)
- new net: LED195.2 (DIN), LED196.4 (DOUT)
- new net: LED195.4 (DOUT), LED199.2 (DIN)
- new net: LED266.4 (DOUT), LED273.2 (DIN)
- new net: LED273.4 (DOUT), LED280.2 (DIN)
- new net: LED324.4 (DOUT), LED331.2 (DIN)
- new net: LED331.4 (DOUT), LED338.2 (DIN)
- new net: LED290.2 (DIN), LED297.4 (DOUT)
- new net: LED290.4 (DOUT), LED291.2 (DIN)
- new net: LED232.2 (DIN), LED239.4 (DOUT)
- new net: LED232.4 (DOUT), LED233.2 (DIN)
- new net: LED259.2 (DIN), LED265.4 (DOUT)
- new net: LED259.4 (DOUT), LED266.2 (DIN)
- new net: LED315.4 (DOUT), LED322.2 (DIN)
- new net: LED322.4 (DOUT), LED329.2 (DIN)
- new net: LED211.2 (DIN), LED218.4 (DOUT)
- new net: LED204.2 (DIN), LED211.4 (DOUT)
- new net: LED200.4 (DOUT), LED201.2 (DIN)
- new net: LED201.4 (DOUT), LED202.2 (DIN)
- new net: LED325.2 (DIN), LED332.4 (DOUT)
- new net: LED318.2 (DIN), LED325.4 (DOUT)
- new net: LED191.4 (DOUT), LED192.2 (DIN)
- new net: LED192.4 (DOUT), LED193.2 (DIN)
- new net: LED329.4 (DOUT), LED336.2 (DIN)
- new net: LED336.4 (DOUT), LED337.2 (DIN)
- new net: LED175.4 (DOUT), LED176.2 (DIN)
- new net: LED176.4 (DOUT), LED177.2 (DIN)
- new net: LED216.2 (DIN), LED223.4 (DOUT)
- new net: LED209.2 (DIN), LED216.4 (DOUT)
- new net: LED177.4 (DOUT), LED178.2 (DIN)
- new net: LED178.4 (DOUT), LED179.2 (DIN)
- new net: LED184.4 (DOUT), LED185.2 (DIN)
- new net: LED185.4 (DOUT), LED186.2 (DIN)
- new net: LED213.2 (DIN), LED220.4 (DOUT)
- new net: LED262.2 (DIN), LED269.4 (DOUT)
- new net: LED262.4 (DOUT), LED263.2 (DIN)
- new net: LED296.4 (DOUT), LED303.2 (DIN)
- new net: LED303.4 (DOUT), LED310.2 (DIN)
- new net: LED267.2 (DIN), LED274.4 (DOUT)
- new net: C212.1, C383.2
- new net: LED304.2 (DIN), LED311.4 (DOUT)
- new net: LED297.2 (DIN), LED304.4 (DOUT)
- new net: LED203.4 (DOUT), LED210.2 (DIN)
- new net: LED210.4 (DOUT), LED217.2 (DIN)
- new net: LED333.4 (DOUT), LED340.2 (DIN)
- new net: LED291.4 (DOUT), LED298.2 (DIN)
- new net: LED248.2 (DIN), LED255.4 (DOUT)
- new net: LED175.2 (DIN), R11.1
- new net: LED334.4 (DOUT), LED341.2 (DIN)
- new net: LED341.4 (DOUT), LED342.2 (DIN)
- new net: LED338.4 (DOUT), LED339.2 (DIN)
- new net: LED239.2 (DIN), LED246.4 (DOUT)
- new net: LED260.2 (DIN), LED267.4 (DOUT)
- new net: LED260.4 (DOUT), LED261.2 (DIN)
- new net: C214.1, C385.2
- new net: LED243.4 (DOUT), LED250.2 (DIN)
- new net: LED250.4 (DOUT), LED257.2 (DIN)
- new net: LED194.4 (DOUT), LED198.2 (DIN)
- new net: D51.2 (A), SW53.2
- new net: LED292.4 (DOUT), LED299.2 (DIN)
- new net: LED299.4 (DOUT), LED306.2 (DIN)
- new net: LED189.2 (DIN), LED190.4 (DOUT)
- new net: LED186.4 (DOUT), LED190.2 (DIN)
- new net: LED236.2 (DIN), R13.1
- new net: LED236.4 (DOUT), LED243.2 (DIN)
- new net: D52.2 (A), SW54.2
- new net: LED298.4 (DOUT), LED305.2 (DIN)
- new net: LED208.4 (DOUT), LED215.2 (DIN)
- new net: LED263.4 (DOUT), LED270.2 (DIN)
- new net: LED235.4 (DOUT), LED242.2 (DIN)
- new net: C211.1, C382.2
- new net: LED218.2 (DIN), LED225.4 (DOUT)
- new net: LED247.4 (DOUT), LED254.2 (DIN)
- new net: LED254.4 (DOUT), LED255.2 (DIN)
- new net: LED251.2 (DIN), LED258.4 (DOUT)
- new net: LED244.2 (DIN), LED251.4 (DOUT)
- new net: LED306.4 (DOUT), LED313.2 (DIN)
- new net: LED313.4 (DOUT), LED314.2 (DIN)
- new net: LED270.4 (DOUT), LED277.2 (DIN)
- new net: LED199.4 (DOUT), LED200.2 (DIN)
- new net: LED332.2 (DIN), LED339.4 (DOUT)
- new net: LED328.2 (DIN), LED335.4 (DOUT)
- new net: LED187.4 (DOUT), LED191.2 (DIN)
- new net: LED317.4 (DOUT), LED324.2 (DIN)
- new net: LED183.4 (DOUT), LED184.2 (DIN)
- new net: LED293.2 (DIN), LED300.4 (DOUT)
- new net: LED287.2 (DIN), LED293.4 (DOUT)
- new net: C213.1, C384.2
- new net: LED272.2 (DIN), LED279.4 (DOUT)
- new net: LED181.4 (DOUT), LED182.2 (DIN)
- new net: LED277.4 (DOUT), LED284.2 (DIN)
- new net: LED320.2 (DIN), R16.1
- new net: LED320.4 (DOUT), LED327.2 (DIN)
- new net: LED330.2 (DIN), LED337.4 (DOUT)
- new net: LED323.2 (DIN), LED330.4 (DOUT)
- new net: LED282.4 (DOUT), LED283.2 (DIN)
- new net: LED276.2 (DIN), LED283.4 (DOUT)
- new net: LED310.4 (DOUT), LED311.2 (DIN)
- new net: LED242.4 (DOUT), LED249.2 (DIN)
- new net: LED249.4 (DOUT), LED256.2 (DIN)
- new net: LED217.4 (DOUT), LED224.2 (DIN)
- new net: LED182.4 (DOUT), LED183.2 (DIN)
- new net: D50.2 (A), SW52.2
- new net: LED269.2 (DIN), LED276.4 (DOUT)
- new net: LED224.4 (DOUT), LED225.2 (DIN)
- new net: LED221.4 (DOUT), LED228.2 (DIN)
- new net: LED288.2 (DIN), LED295.4 (DOUT)
- new net: LED288.4 (DOUT), LED289.2 (DIN)
- new net: LED265.2 (DIN), LED272.4 (DOUT)
- new net: LED289.4 (DOUT), LED296.2 (DIN)
- new net: LED316.2 (DIN), LED323.4 (DOUT)
- new net: LED316.4 (DOUT), LED317.2 (DIN)
- new net: LED203.2 (DIN), LED209.4 (DOUT)
- new net: LED219.4 (DOUT), LED226.2 (DIN)
- new net: LED327.4 (DOUT), LED334.2 (DIN)
- new net: LED257.4 (DOUT), LED258.2 (DIN)
- new net: LED215.4 (DOUT), LED222.2 (DIN)
- new net: LED222.4 (DOUT), LED229.2 (DIN)
- new net: LED261.4 (DOUT), LED268.2 (DIN)
- new net: LED268.4 (DOUT), LED275.2 (DIN)
- new net: LED205.4 (DOUT), LED212.2 (DIN)
- new net: LED212.4 (DOUT), LED219.2 (DIN)
- new net: LED231.2 (DIN), LED237.4 (DOUT)
- new net: LED231.4 (DOUT), LED238.2 (DIN)
- new net: LED292.2 (DIN), R15.1
- new net: LED301.4 (DOUT), LED308.2 (DIN)
- new net: LED238.4 (DOUT), LED245.2 (DIN)
- new net: LED229.4 (DOUT), LED230.2 (DIN)
- new net: C215.1, C386.2
- new net: LED223.2 (DIN), LED230.4 (DOUT)
- new net: LED275.4 (DOUT), LED282.2 (DIN)
- new net: LED204.4 (DOUT), LED205.2 (DIN)
- new net: LED318.4 (DOUT), LED319.2 (DIN)
- new net: LED193.4 (DOUT), LED194.2 (DIN)
- new net: LED287.4 (DOUT), LED294.2 (DIN)
- new net: LED237.2 (DIN), LED244.4 (DOUT)
- new net: LED335.2 (DIN), LED342.4 (DOUT)
- new net: LED294.4 (DOUT), LED301.2 (DIN)
- new net +5V_LED: C100.1, C101.1, C102.1, C103.1, C104.1, C105.1, C106.1, C107.1, C108.1, C109.1, C110.1, C111.1, C112.1, C113.1, C114.1, C115.1, C116.1, C117.1, C118.1, C119.1, C120.1, C121.1, C122.1, C123.1, C124.1, C125.1, C126.1, C127.1, C128.1, C129.1, C130.1, C131.1, C132.1, C133.1, C134.1, C135.1, C136.1, C137.1, C138.1, C139.1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
- new net COL_11: RP2350.14 (GPIO10), SW45.1, SW50.1, SW51.1
- new net COL_12: RP2350.15 (GPIO11), SW52.1, SW53.1, SW54.1
- no-connect marks 10 -> 12
Other:
- note added: "COL_1"
- note added: "COL_2"
- note added: "COL_3"
- note added: "COL_4"
- note added: "COL_5"
- note added: "COL_6"
- note added: "Cirque Trackball"
- note removed: "LED ARRAY"
- moved on the sheet: C65, D11, D44, D45, D46, D47, D6, SW1, SW13, SW46, SW47, SW48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

Commit message: sync
Parts:
- added C38, C39: 100nF, Capacitor_SMD:C_0603_1608Metric, symbol Device:C
- added R38, R39: 10k, Resistor_SMD:R_0603_1608Metric, symbol Device:R
- added U2: LSM6DS3TR-C, easyeda2kicad:LGA-14_L3.0-W2.5-P0.50-TL, symbol easyeda2kicad:LSM6DS3TR-C
- added U3: LSM6DSRTR, easyeda2kicad:LGA-14_L3.0-W2.5-P0.50-BR, symbol easyeda2kicad:LSM6DSRTR
Connections:
- net +3.3V: now also C38.1, C39.1, R39.1, U3.5 (VDDIO), U3.8 (VDD)
- net GND: now also C38.2, C39.2, R38.1, U3.2 (SDX), U3.3 (SCX), U3.6 (GND), U3.7 (GND)
- new net RP2350_GPIO_10: U3.13 (SCL)
- new net RP2350_GPIO_11: U3.14 (SDA)
- new net RP2350_GPIO_5: R38.2, U3.4 (INT1)
- new net RP2350_GPIO_6: U3.9 (INT2)
- new net RP2350_GPIO_7: R39.2, U3.12 (CS)
- new net RP2350_GPIO_8: U3.1 (SDO/SA0)
- no-connect marks 12 -> 14
Other:
- note added: "IMU"
- moved on the sheet: D1, D11, D12, D13, D14, D16, D17, D18, D2, D20, D21, D22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

Commit message: sync
Parts:
- removed C222, C223, C224, C225, C226, C38, C39: 100nF, Capacitor_SMD:C_0603_1608Metric, symbol Device:C
- removed C383, C384, C385, C386, C387: 100nF, Capacitor_SMD:C_0402_1005Metric, symbol Device:C
- removed R38, R39: 10k, Resistor_SMD:R_0603_1608Metric, symbol Device:R
- removed U1: SN74LVC8T245, symbol Logic_LevelTranslator:SN74LVC8T245
- removed U3: LSM6DSRTR, easyeda2kicad:LGA-14_L3.0-W2.5-P0.50-BR, symbol easyeda2kicad:LSM6DSRTR
- added FPC1: FPC-05F-12PH20, easyeda2kicad:FPC-SMD_12P-P0.50_FPC-05F-12PH20, symbol easyeda2kicad:FPC-05F-12PH20
- added R40, R41: 4.7k, Resistor_SMD:R_0402_1005Metric, symbol Device:R
- added U6: SN74LVC1T45DBVR, easyeda2kicad:SOT-23-6_L2.9-W1.6-P0.95-LS2.8-BR, symbol easyeda2kicad:SN74LVC1T45DBVR
- C212, C213, C214, C215, C216: value 22uF -> 100nF; footprint Capacitor_SMD:C_0402_1005Metric -> Capacitor_SMD:C_0603_1608Metric
Connections:
- net 5V_A3 is gone; now on net SD_CS: RP2350.29 (GPIO18)
- net 5V_A4 is gone; now on net SPI_SCK: RP2350.31 (GPIO19)
- net 5V_A5 is gone; now on net SPI_MOSI: RP2350.32 (GPIO20)
- net 5V_A6 is gone; now on net SPI_MISO: RP2350.33 (GPIO21)
- net RP2350_GPIO_22 is gone; now on net IMU_INT1: RP2350.34 (GPIO22)
- net RP2350_GPIO_24 is gone; now on net I2C_SDA: RP2350.36 (GPIO24)
- net RP2350_GPIO_25 is gone; now on net I2C_SCL: RP2350.37 (GPIO25)
- net RP2350_GPIO_26_ADC is gone; now on net ENC_A: RP2350.40 (GPIO26/ADC0)
- net RP2350_GPIO_27_ADC is gone; now on net ENC_B: RP2350.41 (GPIO27/ADC1)
- net RP2350_GPIO_28_ADC is gone; now on net ENC_SW: RP2350.42 (GPIO28/ADC2)
- net RP2350_GPIO_29_ADC is gone; now on net IMU_CS: RP2350.43 (GPIO29/ADC3)
- net +3.3V: now also LED1.2 (VDD), U2.5 (VDDIO), U2.8 (VDD), FPC1.12, R40.1, R41.1, U6.1 (VCCA), U6.5 (DIR)
- net +5V_LED: now also C212.1, C213.1, C214.1, C215.1, C216.1, LED187.3 (VDD), LED204.3 (VDD), LED232.3 (VDD), LED260.3 (VDD), LED288.3 (VDD), LED316.3 (VDD), U6.6 (VCCB)
- net COL_1: no longer R11.2, R12.2, R13.2, R14.2, R15.2, R16.2
- net GND: now also LED1.3 (GND), SW1.6, SW1.7, SW1.C, SW1.E, U2.2 (SDx), U2.3 (SCx), U2.6 (GND), U2.7 (GND), FPC1.11, FPC1.13, FPC1.14, U6.2 (GND)
- net SPI_MISO: now also U2.1 (SDO/SA0)
- net SPI_MOSI: now also U2.14 (SDA)
- net SPI_SCK: now also U2.13 (SCL)
- net LEDA_L1: now reaches LED312.4 (DOUT)
- net LEDA_L1: now also LED202.4 (DOUT), LED228.4 (DOUT), LED256.4 (DOUT), LED284.4 (DOUT), LED340.4 (DOUT)
- net ENC_A: now reaches SW1.A
- net ENC_B: now reaches SW1.B
- net ENC_SW: now reaches SW1.D
- net IMU_CS: now reaches U2.12 (CS)
- net IMU_INT1: now reaches U2.4 (INT1)
- net I2C_SCL: now reaches LED1.1 (SCL)
- net I2C_SCL: now also FPC1.9, R41.2
- net I2C_SDA: now reaches LED1.4 (SDA)
- net I2C_SDA: now also FPC1.10, R40.2
- net 5V_A1 renamed LED_DATA
- net LED_DATA: now also U6.3 (A)
- net 5V_A2 renamed TP_DR
- net TP_DR: now also FPC1.4
- net RP2350_GPIO_23 renamed STATUS
- new net LED_DIN_A: R11.2, R12.2, R13.2, R14.2, R15.2, R16.2, U6.4 (B)
- no-connect marks 14 -> 20
Other:
- note removed: "COL_1"
- note removed: "COL_2"
- note removed: "COL_3"
- note removed: "COL_4"
- note removed: "COL_5"
- note removed: "COL_6"
- moved on the sheet: C301, C65, LED1, U12, U2

Commit message: sync
Parts:
- added C400: 10uF, Capacitor_SMD:C_0805_2012Metric, symbol Device:C
- added C401: 100uF, Capacitor_SMD:C_1206_3216Metric, symbol Device:C
- added F1: 500mA, Fuse:Fuse_1206_3216Metric, symbol Device:Polyfuse
- added FB1: Ferrite 600R@100MHz, Inductor_SMD:L_0805_2012Metric, symbol Device:L
Connections:
- net +3.3V: now also C4.2, R6.1, RP2350.46 (VREG_AVDD)
- net +5V_LED: now also C401.1, FB1.2
- net GND: now also C400.2, C401.2
- net USB_VBUS: now also F1.1
- net BATT_SW+ renamed +5V
- net +5V: now also C400.1, F1.2, FB1.1
- no-connect marks 20 -> 21
Other:
- moved on the sheet: Card1, R28, R29, R30, R31, R36, R37

Commit message: sync
Parts:
- removed D47: D, symbol Device:D
- removed SW49: SW_Push, symbol Switch:SW_Push
- added LED2: SK6805-EC15, easyeda2kicad:LED-SMD_4P-L1.5-W1.5-BL, symbol easyeda2kicad:SK6805-EC15
- D1, D11, D12, D13, D14, D16, D17, D18, D2, D20, D21, D22, D24, D25, D26, D28, D29, D3, D30, D32, D33, D34, D36, D37, D38, D40, D41, D42, D43, D44, D45, D46, D48, D49, D50, D51, D52, D6, D7, D8, D9: footprint (none) -> Diode_SMD:D_0603_1608Metric
- SW10, SW11, SW13, SW14, SW15, SW16, SW18, SW19, SW20, SW22, SW23, SW24, SW26, SW27, SW28, SW30, SW31, SW32, SW34, SW35, SW36, SW38, SW39, SW4, SW40, SW42, SW43, SW44, SW45, SW46, SW47, SW48, SW5, SW50, SW51, SW52, SW53, SW54, SW6, SW9: footprint (none) -> PCM_Switch_Keyboard_Hotswap_Kailh:SW_Hotswap_Kailh_Choc_V1V2_1.00u
- SW8: footprint (none) -> PCM_Switch_Keyboard_Hotswap_Kailh:SW_Hotswap_Kailh_Choc_V1V2_2.00u

Commit message: sync
Parts:
- removed C202, C203, C204, C205, C206, C207, C208, C209, C210, C212, C213, C214, C215, C216, C217, C218, C219, C220, C221, C49, C50, C51, C52, C53, C54, C55, C56, C57, C58, C59, C60, C61, C66, C67, C68, C69, C70, C71, C72, C73, C74, C75, C76, C77, C78, C79, C80, C81: 100nF, Capacitor_SMD:C_0603_1608Metric, symbol Device:C
- removed LED175, LED176, LED177, LED178, LED179, LED180, LED181, LED182, LED183, LED184, LED185, LED186, LED187, LED188, LED189, LED190, LED191, LED192, LED193, LED194, LED195, LED196, LED197, LED198, LED199, LED200, LED201, LED202, LED203, LED204, LED205, LED206, LED207, LED208, LED209, LED210, LED211, LED212, LED213, LED214, LED215, LED216, LED217, LED218, LED219, LED220, LED221, LED222, LED223, LED224, LED225, LED226, LED227, LED228, LED229, LED230, LED231, LED232, LED233, LED234, LED235, LED236, LED237, LED238, LED239, LED240, LED241, LED242, LED243, LED244, LED245, LED246, LED247, LED248, LED249, LED250, LED251, LED252, LED253, LED254, LED255, LED256, LED257, LED258, LED259, LED260, LED261, LED262, LED263, LED264, LED265, LED266, LED267, LED268, LED269, LED270, LED271, LED272, LED273, LED274, LED275, LED276, LED277, LED278, LED279, LED280, LED281, LED282, LED283, LED284, LED285, LED286, LED287, LED288, LED289, LED290, LED291, LED292, LED293, LED294, LED295, LED296, LED297, LED298, LED299, LED300, LED301, LED302, LED303, LED304, LED305, LED306, LED307, LED308, LED309, LED310, LED311, LED312, LED313, LED314, LED315, LED316, LED317, LED318, LED319, LED320, LED321, LED322, LED323, LED324, LED325, LED326, LED327, LED328, LED329, LED330, LED331, LED332, LED333, LED334, LED335, LED336, LED337, LED338, LED339, LED340, LED341, LED342, STATUS1: SK6812MINI-E_C5149201, easyeda2kicad:LED-SMD_4P-L3.2-W2.8-LS5.9_SK6812MINI-E, symbol easyeda2kicad:SK6812MINI-E_C5149201
- removed R11, R12, R14, R15, R16: 470, Resistor_SMD:R_0603_1608Metric, symbol Device:R
- added C383, C384, C385, C386, C387, C388, C389, C390, C391, C392, C393, C394, C395, C396, C397, C398, C399, C402, C403, C404, C405, C406, C407, C408, C409, C410, C411, C412, C413, C414, C415, C416, C417, C418, C419, C420, C421, C422, C423, C424: 100nF, Capacitor_SMD:C_0402_1005Metric, symbol Device:C
- added J2: Conn_01x05_Pin, Connector_PinHeader_2.54mm:PinHeader_1x05_P2.54mm_Vertical, symbol Connector:Conn_01x05_Pin
- added J3: Conn_01x04_Pin, Connector_PinHeader_2.54mm:PinHeader_1x04_P2.54mm_Vertical, symbol Connector:Conn_01x04_Pin
- added LED10, LED100, LED101, LED102, LED103, LED104, LED105, LED106, LED107, LED108, LED109, LED11, LED110, LED111, LED112, LED113, LED114, LED115, LED116, LED117, LED118, LED119, LED12, LED120, LED121, LED122, LED13, LED14, LED15, LED16, LED17, LED18, LED19, LED20, LED21, LED22, LED23, LED24, LED25, LED26, LED27, LED28, LED29, LED3, LED30, LED31, LED32, LED33, LED34, LED35, LED36, LED37, LED38, LED39, LED4, LED40, LED41, LED42, LED43, LED44, LED45, LED46, LED47, LED48, LED49, LED5, LED50, LED51, LED52, LED53, LED54, LED55, LED56, LED57, LED58, LED59, LED6, LED60, LED61, LED62, LED63, LED64, LED65, LED66, LED67, LED68, LED69, LED7, LED70, LED71, LED72, LED73, LED74, LED75, LED76, LED77, LED78, LED79, LED8, LED80, LED81, LED82, LED83, LED84, LED85, LED86, LED87, LED88, LED89, LED9, LED90, LED91, LED92, LED93, LED94, LED95, LED96, LED97, LED98, LED99: SK6805-EC15, easyeda2kicad:LED-SMD_4P-L1.5-W1.5-BL, symbol easyeda2kicad:SK6805-EC15
- added U1, U10, U11, U13, U14, U15, U16, U17, U19, U20, U21, U22, U23, U24, U25, U26, U27, U28, U29, U30, U31, U32, U33, U34, U35, U36, U37, U38, U39, U4, U40, U41, U42, U44, U45, U46, U47, U5, U7, U8, U9: CH604ASR, easyeda2kicad:SOT-23-3_L2.9-W1.6-P1.90-LS2.8-BR, symbol easyeda2kicad:CH604ASR
- added U18, U3, U43: CD74HC4067SM, Package_SO:SSOP-24_5.3x8.2mm_P0.65mm, symbol 74xx:CD74HC4067SM
- D1, D11, D12, D13, D14, D16, D17, D18, D2, D20, D21, D22, D24, D25, D26, D28, D29, D3, D30, D32, D33, D34, D36, D37, D38, D40, D41, D42, D43, D44, D45, D46, D48, D49, D50, D51, D52, D6, D7, D8, D9: now not fitted; now left out of the parts list
- SW10, SW11, SW13, SW14, SW15, SW16, SW18, SW19, SW20, SW22, SW23, SW24, SW26, SW27, SW28, SW30, SW31, SW32, SW34, SW35, SW36, SW38, SW39, SW4, SW40, SW42, SW43, SW44, SW45, SW46, SW47, SW48, SW5, SW50, SW51, SW52, SW53, SW54, SW6, SW9: footprint PCM_Switch_Keyboard_Hotswap_Kailh:SW_Hotswap_Kailh_Choc_V1V2_1.00u -> PCM_Switch_Keyboard_Cherry_MX:SW_Cherry_MX_PCB
- SW8: footprint PCM_Switch_Keyboard_Hotswap_Kailh:SW_Hotswap_Kailh_Choc_V1V2_2.00u -> PCM_Switch_Keyboard_Cherry_MX:SW_Cherry_MX_PCB
Connections:
- net +3.3V: now also C383.1, C384.1, C385.1, C386.1, C387.1, C388.1, C389.1, C390.1, C391.1, C392.1, C393.1, C394.1, C395.1, C396.1, C397.1, C398.1, C399.1, C402.1, C403.1, C404.1, C405.1, C406.1, C407.1, C408.1, C409.1, C410.1, C411.1, C412.1, C413.1, C414.1, C415.1, C416.1, C417.1, C418.1, C419.1, C420.1, C421.1, C422.1, C423.1, C424.1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; no longer C4.2, R6.1, RP2350.46 (VREG_AVDD)
- net +5V_LED: now also LED2.2 (VDD), LED10.2 (VDD), LED100.2 (VDD), LED101.2 (VDD), LED102.2 (VDD), LED103.2 (VDD), LED104.2 (VDD), LED105.2 (VDD), LED106.2 (VDD), LED107.2 (VDD), LED108.2 (VDD), LED109.2 (VDD), LED11.2 (VDD), LED110.2 (VDD), LED111.2 (VDD), LED112.2 (VDD), LED113.2 (VDD), LED114.2 (VDD), LED115.2 (VDD), LED116.2 (VDD), LED117.2 (VDD), LED118.2 (VDD), LED119.2 (VDD), LED12.2 (VDD), LED120.2 (VDD), LED121.2 (VDD), LED13.2 (VDD), LED14.2 (VDD), LED15.2 (VDD), LED16.2 (VDD), LED17.2 (VDD), LED18.2 (VDD), LED19.2 (VDD), LED20.2 (VDD), LED21.2 (VDD), LED22.2 (VDD), LED23.2 (VDD), LED24.2 (VDD), LED25.2 (VDD), LED26.2 (VDD)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
- net COL_1: no longer RP2350.2 (GPIO0)
- net COL_10: no longer RP2350.13 (GPIO9)
- net COL_11: no longer RP2350.14 (GPIO10)
- net COL_12: no longer RP2350.15 (GPIO11)
- net COL_2: no longer RP2350.3 (GPIO1)
- net COL_3: no longer RP2350.4 (GPIO2)
- net COL_4: no longer RP2350.5 (GPIO3)
- net COL_5: no longer RP2350.7 (GPIO4)
- net COL_6: no longer RP2350.8 (GPIO5)
- net COL_7: no longer RP2350.9 (GPIO6)
- net COL_8: no longer RP2350.10 (GPIO7)
- net COL_9: no longer RP2350.12 (GPIO8)
- net ENC_A: now also RP2350.7 (GPIO4); no longer RP2350.40 (GPIO26/ADC0)
- net ENC_B: now also RP2350.8 (GPIO5); no longer RP2350.41 (GPIO27/ADC1)
- net ENC_SW: now also RP2350.9 (GPIO6); no longer RP2350.42 (GPIO28/ADC2)
- net GND: now also LED2.4 (GND), C383.2, C384.2, C385.2, C386.2, C387.2, C388.2, C389.2, C390.2, C391.2, C392.2, C393.2, C394.2, C395.2, C396.2, C397.2, C398.2, C399.2, C402.2, C403.2, C404.2, C405.2, C406.2, C407.2, C408.2, C409.2, C410.2, C411.2, C412.2, C413.2, C414.2, C415.2, C416.2, C417.2, C418.2, C419.2, C420.2, C421.2, C422.2, C423.2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
- net ROW_1: no longer RP2350.16 (GPIO12)
- net ROW_2: no longer RP2350.17 (GPIO13)
- net ROW_3: no longer RP2350.18 (GPIO14)
- net ROW_4: no longer RP2350.19 (GPIO15)
- net at R10.1: now also LED122.1 (DIN)
- net at R13.1: now also LED2.1 (DIN)
- net at LED2.3 (DOUT): now also LED3.1 (DIN)
- new net: LED29.1 (DIN), LED46.3 (DOUT)
- new net: LED29.3 (DOUT), LED35.1 (DIN)
- new net: LED107.3 (DOUT), LED113.1 (DIN)
- new net: LED113.3 (DOUT), LED119.1 (DIN)
- new net: LED35.3 (DOUT), LED41.1 (DIN)
- new net: LED41.3 (DOUT), LED47.1 (DIN)
- new net: U41.2 (OUT), U43.2 (I7)
- new net: U43.20 (I11), U47.2 (OUT)
- new net: U43.21 (I10), U46.2 (OUT)
- new net: U43.22 (I9), U45.2 (OUT)
- new net: U42.2 (OUT), U43.23 (I8)
- new net: U40.2 (OUT), U43.3 (I6)
- new net: U39.2 (OUT), U43.4 (I5)
- new net: U38.2 (OUT), U43.5 (I4)
- new net: U37.2 (OUT), U43.6 (I3)
- new net: U36.2 (OUT), U43.7 (I2)
- new net: U35.2 (OUT), U43.8 (I1)
- new net: U34.2 (OUT), U43.9 (I0)
- new net: LED67.3 (DOUT), LED73.1 (DIN)
- new net: LED51.1 (DIN), LED73.3 (DOUT)
- new net: LED43.3 (DOUT), LED49.1 (DIN)
- new net: LED25.1 (DIN), LED49.3 (DOUT)
- new net: LED106.3 (DOUT), LED112.1 (DIN)
- new net: LED112.3 (DOUT), LED118.1 (DIN)
- new net: LED45.3 (DOUT), LED50.1 (DIN)
- new net: LED50.3 (DOUT), LED56.1 (DIN)
- new net: LED40.3 (DOUT), LED46.1 (DIN)
- new net: U1.2 (OUT), U3.9 (I0)
- new net: LED79.3 (DOUT), LED85.1 (DIN)
- new net: LED85.3 (DOUT), LED91.1 (DIN)
- new net: U18.5 (I4), U23.2 (OUT)
- new net: LED15.3 (DOUT), LED17.1 (DIN)
- new net: LED17.3 (DOUT), LED19.1 (DIN)
- new net: U18.18 (I13), U32.2 (OUT)
- new net: LED4.3 (DOUT), LED5.1 (DIN)
- new net: LED5.3 (DOUT), LED6.1 (DIN)
- new net: LED16.3 (DOUT), LED18.1 (DIN)
- new net: LED18.3 (DOUT), LED20.1 (DIN)
- new net: LED60.3 (DOUT), LED66.1 (DIN)
- new net: LED66.3 (DOUT), LED72.1 (DIN)
- new net: LED52.1 (DIN), LED68.3 (DOUT)
- new net: LED52.3 (DOUT), LED58.1 (DIN)
- new net: U11.2 (OUT), U3.2 (I7)
- new net: LED55.1 (DIN), LED72.3 (DOUT)
- new net: LED39.3 (DOUT), LED45.1 (DIN)
- new net: LED78.3 (DOUT), LED84.1 (DIN)
- new net: LED84.3 (DOUT), LED90.1 (DIN)
- new net: U18.22 (I9), U28.2 (OUT)
- new net: LED21.3 (DOUT), LED22.1 (DIN)
- new net: LED22.3 (DOUT), LED24.1 (DIN)
- new net: LED87.3 (DOUT), LED93.1 (DIN)
- new net: LED93.3 (DOUT), LED98.1 (DIN)
- new net: LED103.1 (DIN), LED120.3 (DOUT)
- new net: LED103.3 (DOUT), LED109.1 (DIN)
- new net: LED7.3 (DOUT), LED8.1 (DIN)
- new net: LED8.3 (DOUT), LED9.1 (DIN)
- new net: U10.2 (OUT), U3.3 (I6)
- new net: U18.17 (I14), U33.2 (OUT)
- new net: U18.2 (I7), U26.2 (OUT)
- new net: LED36.3 (DOUT), LED42.1 (DIN)
- new net: LED42.3 (DOUT), LED48.1 (DIN)
- new net: LED79.1 (DIN), LED96.3 (DOUT)
- new net: LED51.3 (DOUT), LED57.1 (DIN)
- new net: J3.1 (Pin_1), RP2350.19 (GPIO15)
- new net: J3.2 (Pin_2), RP2350.18 (GPIO14)
- new net: J3.3 (Pin_3), RP2350.17 (GPIO13)
- new net: J3.4 (Pin_4), RP2350.16 (GPIO12)
- new net: U18.8 (I1), U20.2 (OUT)
- new net: LED89.3 (DOUT), LED95.1 (DIN)
- new net: LED78.1 (DIN), LED95.3 (DOUT)
- new net: LED75.1 (DIN), LED97.3 (DOUT)
- new net: LED75.3 (DOUT), LED81.1 (DIN)
- new net: U18.6 (I3), U22.2 (OUT)
- new net: LED25.3 (DOUT), LED33.1 (DIN)
- new net: LED105.3 (DOUT), LED111.1 (DIN)
- new net: LED111.3 (DOUT), LED117.1 (DIN)
- new net: LED101.1 (DIN), LED118.3 (DOUT)
- new net: U18.23 (I8), U27.2 (OUT)
- new net: LED83.3 (DOUT), LED89.1 (DIN)
- new net: LED24.3 (DOUT), LED26.1 (DIN)
- new net: LED91.3 (DOUT), LED97.1 (DIN)
- new net: LED86.3 (DOUT), LED92.1 (DIN)
- new net: LED76.1 (DIN), LED92.3 (DOUT)
- new net: U3.8 (I1), U4.2 (OUT)
- new net: LED38.3 (DOUT), LED44.1 (DIN)
- new net: LED27.1 (DIN), LED44.3 (DOUT)
- new net: LED6.3 (DOUT), LED7.1 (DIN)
- new net: U16.2 (OUT), U3.20 (I11)
- new net: LED61.3 (DOUT), LED67.1 (DIN)
- new net: U14.2 (OUT), U3.22 (I9)
- new net: LED53.3 (DOUT), LED59.1 (DIN)
- new net: LED59.3 (DOUT), LED65.1 (DIN)
- new net: LED102.1 (DIN), LED119.3 (DOUT)
- new net: LED102.3 (DOUT), LED108.1 (DIN)
- new net: LED19.3 (DOUT), LED21.1 (DIN)
- new net: LED90.3 (DOUT), LED96.1 (DIN)
- new net: LED108.3 (DOUT), LED114.1 (DIN)
- new net: LED114.3 (DOUT), LED120.1 (DIN)
- new net: LED100.1 (DIN), LED116.3 (DOUT)
- new net: LED100.3 (DOUT), LED106.1 (DIN)
- new net: LED58.3 (DOUT), LED64.1 (DIN)
- new net: U3.7 (I2), U5.2 (OUT)
- new net: LED31.1 (DIN), LED48.3 (DOUT)
- new net: LED69.3 (DOUT), LED74.1 (DIN)
- new net: LED74.3 (DOUT), LED80.1 (DIN)
- new net: LED115.3 (DOUT), LED121.1 (DIN)
- new net: LED121.3 (DOUT), LED99.1 (DIN)
- new net: LED88.3 (DOUT), LED94.1 (DIN)
- new net: LED77.1 (DIN), LED94.3 (DOUT)
- new net: J2.1 (Pin_1), RP2350.15 (GPIO11)
- new net: J2.2 (Pin_2), RP2350.14 (GPIO10)
- new net: J2.3 (Pin_3), RP2350.13 (GPIO9)
- new net: J2.4 (Pin_4), RP2350.12 (GPIO8)
- new net: J2.5 (Pin_5), RP2350.10 (GPIO7)
- new net: LED26.3 (DOUT), LED28.1 (DIN)
- new net: LED82.3 (DOUT), LED88.1 (DIN)
- new net: LED27.3 (DOUT), LED34.1 (DIN)
- new net: LED34.3 (DOUT), LED40.1 (DIN)
- new net: U17.2 (OUT), U3.19 (I12)
- new net: LED105.1 (DIN), LED99.3 (DOUT)
- new net: LED10.1 (DIN), LED9.3 (DOUT)
- new net: LED10.3 (DOUT), LED11.1 (DIN)
- new net: LED81.3 (DOUT), LED87.1 (DIN)
- new net: U18.4 (I5), U24.2 (OUT)
- new net: LED14.3 (DOUT), LED16.1 (DIN)
- new net: LED57.3 (DOUT), LED63.1 (DIN)
- new net: LED109.3 (DOUT), LED115.1 (DIN)
- new net: U3.5 (I4), U8.2 (OUT)
- new net: LED101.3 (DOUT), LED107.1 (DIN)
- new net: U15.2 (OUT), U3.21 (I10)
- new net: U13.2 (OUT), U3.23 (I8)
- new net: U3.4 (I5), U9.2 (OUT)
- new net: U3.6 (I3), U7.2 (OUT)
- new net: LED3.3 (DOUT), LED4.1 (DIN)
- new net: C4.2, R6.1, RP2350.46 (VREG_AVDD)
- new net: U18.7 (I2), U21.2 (OUT)
- new net: LED30.3 (DOUT), LED36.1 (DIN)
- new net: LED63.3 (DOUT), LED69.1 (DIN)
- new net: LED80.3 (DOUT), LED86.1 (DIN)
- new net: LED55.3 (DOUT), LED61.1 (DIN)
- new net: LED104.1 (DIN), LED98.3 (DOUT)
- new net: LED104.3 (DOUT), LED110.1 (DIN)
- new net: LED110.3 (DOUT), LED116.1 (DIN)
- new net: LED23.3 (DOUT), LED32.1 (DIN)
- new net: LED32.3 (DOUT), LED38.1 (DIN)
- new net: LED30.1 (DIN), LED47.3 (DOUT)
- new net: LED77.3 (DOUT), LED83.1 (DIN)
- new net: LED56.3 (DOUT), LED62.1 (DIN)
- new net: LED23.1 (DIN), LED28.3 (DOUT)
- new net: U18.20 (I11), U30.2 (OUT)
- new net: LED62.3 (DOUT), LED68.1 (DIN)
- new net: LED65.3 (DOUT), LED71.1 (DIN)
- new net: LED11.3 (DOUT), LED12.1 (DIN)
- new net: LED76.3 (DOUT), LED82.1 (DIN)
- new net: U18.21 (I10), U29.2 (OUT)
- new net: LED64.3 (DOUT), LED70.1 (DIN)
- new net: U18.3 (I6), U25.2 (OUT)
- new net: U18.16 (I15), U44.2 (OUT)
- new net: U18.19 (I12), U31.2 (OUT)
- new net: U18.9 (I0), U19.2 (OUT)
- new net: LED53.1 (DIN), LED70.3 (DOUT)
- new net: LED12.3 (DOUT), LED13.1 (DIN)
- new net: LED15.1 (DIN), LED20.3 (DOUT)
- new net: LED54.3 (DOUT), LED60.1 (DIN)
- new net: LED13.3 (DOUT), LED14.1 (DIN)
- new net: LED37.3 (DOUT), LED43.1 (DIN)
- new net: LED31.3 (DOUT), LED37.1 (DIN)
- new net: LED33.3 (DOUT), LED39.1 (DIN)
- new net: LED54.1 (DIN), LED71.3 (DOUT)
- new net MUX_1: RP2350.40 (GPIO26/ADC0), U3.1 (COM)
- new net MUX_2: RP2350.41 (GPIO27/ADC1), U18.1 (COM)
- new net MUX_3: RP2350.42 (GPIO28/ADC2), U43.1 (COM)
- new net MUX_S0: RP2350.2 (GPIO0), U18.10 (S0), U3.10 (S0), U43.10 (S0)
- new net MUX_S1: RP2350.3 (GPIO1), U18.11 (S1), U3.11 (S1), U43.11 (S1)
- new net MUX_S2: RP2350.4 (GPIO2), U18.14 (S2), U3.14 (S2), U43.14 (S2)
- new net MUX_S3: RP2350.5 (GPIO3), U18.13 (S3), U3.13 (S3), U43.13 (S3)
Other:
- note added: "Keyboard Hall-Effect Sensors"
- moved on the sheet: C400, C401, F1, FB1, LED2, R10, SW10, SW11, SW13, SW14, SW15, SW16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
