File: Atrium PCB/Atrium PCB.kicad_sch (KiCad schematic)
At the start: 1078 parts, among them J1 Conn_01x05_Pin, SW1 EC11E09244BS, SW10 SW_Push, SW11 SW_Push, SW13 SW_Push, SW14 SW_Push, SW15 SW_Push, SW16 SW_Push, SW18 SW_Push, SW19 SW_Push, SW2 SKRPACE010, SW20 SW_Push, SW22 SW_Push, SW23 SW_Push, SW24 SW_Push, SW26 SW_Push, SW27 SW_Push, SW28 SW_Push, SW3 SKRPACE010, SW30 SW_Push, SW31 SW_Push, SW32 SW_Push, SW34 SW_Push, SW35 SW_Push, SW36 SW_Push, SW38 SW_Push, SW39 SW_Push, SW4 SW_Push, SW40 SW_Push, SW41 FG-TC-12E-02-8H, SW42 SW_Push, SW43 SW_Push, SW44 SW_Push, SW45 SW_Push, SW46 SW_Push, SW47 SW_Push, SW48 SW_Push, SW49 FG-TC-12E-02-8H, SW5 SW_Push, SW50 SW_Push, SW51 SW_Push, SW52 SW_Push, SW53 SW_Push, SW54 SW_Push, SW55 FG-TC-12E-02-8H, SW56 FG-TC-12E-02-8H, SW57 FG-TC-12E-02-8H, SW58 FG-TC-12E-02-8H, SW59 FG-TC-12E-02-8H, SW6 SW_Push, SW60 FG-TC-12E-02-8H, SW8 SW_Push, SW9 SW_Push, U1 CH604ASR, U10 CH604ASR, U11 CH604ASR, U12 AP2112K-3.3, U13 CH604ASR, U14 CH604ASR, U15 CH604ASR, U16 CH604ASR, U17 CH604ASR, U18 CD74HC4067SM, U19 CH604ASR, U2 LSM6DS3TR-C, U20 CH604ASR, U21 CH604ASR, U22 CH604ASR, U23 CH604ASR, U24 CH604ASR, U25 CH604ASR, U26 CH604ASR, U27 CH604ASR, U28 CH604ASR, U29 CH604ASR, U3 CD74HC4067SM, U30 CH604ASR, U31 CH604ASR, U32 CH604ASR, U33 CH604ASR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

Commit message: sync
Parts:
- added C25, C26: 100nF, Capacitor_SMD:C_0603_1608Metric, symbol Device:C
- added C545, C546, C547, C548: 100nF, Capacitor_SMD:C_0402_1005Metric, symbol Device:C
- added LED54: SK6805-EC15, easyeda2kicad:LED-SMD_4P-L1.5-W1.5-BL, symbol easyeda2kicad:SK6805-EC15
Connections:
- net +3.3V: now also C25.1, C26.1, C545.1, C546.1, C547.1, C548.1, LED54.2 (VDD)
- net GND: now also C25.2, C26.2, C545.2, C546.2, C547.2, C548.2, LED54.4 (GND)
- net at R10.1: now also LED54.1 (DIN)
Other:
- moved on the sheet: C413, C414, C415

Commit message: sync
Parts:
- removed C513, C532, C544: 100nF, Capacitor_SMD:C_0603_1608Metric, symbol Device:C
- removed LED423, LED461, LED465: SK6805-EC15, easyeda2kicad:LED-SMD_4P-L1.5-W1.5-BL, symbol easyeda2kicad:SK6805-EC15
Connections:
- net LED_DATA: now also RP2350.27 (GPIO16); no longer RP2350.28 (GPIO17)
- net SD_CD: now also RP2350.28 (GPIO17)
- net at LED453.3 (DOUT): now also LED477.1 (DIN)
