File: Atrium PCB/Atrium PCB.kicad_sch (KiCad schematic)
At the start: 1079 parts, among them J1 Conn_01x05_Pin, SW1 EC11E09244BS, SW10 SW_Push, SW11 SW_Push, SW13 SW_Push, SW14 SW_Push, SW15 SW_Push, SW16 SW_Push, SW18 SW_Push, SW19 SW_Push, SW2 SKRPACE010, SW20 SW_Push, SW22 SW_Push, SW23 SW_Push, SW24 SW_Push, SW26 SW_Push, SW27 SW_Push, SW28 SW_Push, SW3 SKRPACE010, SW30 SW_Push, SW31 SW_Push, SW32 SW_Push, SW34 SW_Push, SW35 SW_Push, SW36 SW_Push, SW38 SW_Push, SW39 SW_Push, SW4 SW_Push, SW40 SW_Push, SW41 FG-TC-12E-02-8H, SW42 SW_Push, SW43 SW_Push, SW44 SW_Push, SW45 SW_Push, SW46 SW_Push, SW47 SW_Push, SW48 SW_Push, SW49 FG-TC-12E-02-8H, SW5 SW_Push, SW50 SW_Push, SW51 SW_Push, SW52 SW_Push, SW53 SW_Push, SW54 SW_Push, SW55 FG-TC-12E-02-8H, SW56 FG-TC-12E-02-8H, SW57 FG-TC-12E-02-8H, SW58 FG-TC-12E-02-8H, SW59 FG-TC-12E-02-8H, SW6 SW_Push, SW60 FG-TC-12E-02-8H, SW8 SW_Push, SW9 SW_Push, U1 CH604ASR, U10 CH604ASR, U11 CH604ASR, U12 AP2112K-3.3, U13 CH604ASR, U14 CH604ASR, U15 CH604ASR, U16 CH604ASR, U17 CH604ASR, U18 CD74HC4067SM, U19 CH604ASR, U2 LSM6DS3TR-C, U20 CH604ASR, U21 CH604ASR, U22 CH604ASR, U23 CH604ASR, U24 CH604ASR, U25 CH604ASR, U26 CH604ASR, U27 CH604ASR, U28 CH604ASR, U29 CH604ASR, U3 CD74HC4067SM, U30 CH604ASR, U31 CH604ASR, U32 CH604ASR, U33 CH604ASR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

Commit message: sync
Connections:
- net at U43.16 (I15): now also U31.2 (OUT)
- net at U43.17 (I14): now also U32.2 (OUT)
- net at U43.18 (I13): now also U33.2 (OUT)
- net at U43.19 (I12): now also U44.2 (OUT)
- net at U18.18 (I13): no longer U32.2 (OUT)
- net at U18.17 (I14): no longer U33.2 (OUT)
- net at U18.16 (I15): no longer U44.2 (OUT)
- net at U18.19 (I12): no longer U31.2 (OUT)
Changed lines of the file:
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@@
 	(wire
 		(pts
+			(xy 844.55 201.93) (xy 614.68 201.93)
+		)
+		(stroke
+			(width 0)
+			(type default)
+		)
+	)
+	(wire
+		(pts
 			(xy 57.15 746.76) (xy 60.96 746.76)
 		)
@@
 	(wire
 		(pts
-			(xy 847.09 156.21) (xy 595.63 156.21)
-		)
-		(stroke
-			(width 0)
-			(type default)
-		)
-	)
-	(wire
-		(pts
 			(xy 720.09 435.61) (xy 867.41 435.61)
 		)
@@
 	(wire
 		(pts
-			(xy 844.55 153.67) (xy 595.63 153.67)
-		)
-		(stroke
-			(width 0)
-			(type default)
-		)
-	)
-	(wire
-		(pts
 			(xy 822.96 607.06) (xy 826.77 607.06)
 		)
@@
 	(wire
 		(pts
-			(xy 839.47 55.88) (xy 839.47 148.59)
+			(xy 839.47 55.88) (xy 839.47 207.01)
 		)
 		(stroke
@@
 	(wire
 		(pts
+			(xy 839.47 207.01) (xy 614.68 207.01)
+		)
+		(stroke
+			(width 0)
+			(type default)
+		)
+	)
+	(wire
+		(pts
 			(xy 367.03 525.78) (xy 367.03 515.62)
 		)
@@
 	(wire
 		(pts
+			(xy 842.01 204.47) (xy 614.68 204.47)
+		)
+		(stroke
+			(width 0)
+			(type default)
+		)
+	)
+	(wire
+		(pts
 			(xy 29.21 712.47) (xy 29.21 702.31)
 		)
@@
 	(wire
 		(pts
+			(xy 847.09 199.39) (xy 614.68 199.39)
+		)
+		(stroke
+			(width 0)
+			(type default)
+		)
+	)
+	(wire
+		(pts
 			(xy 554.99 138.43) (xy 570.23 138.43)
 		)
@@
 	(wire
 		(pts
-			(xy 844.55 83.82) (xy 844.55 153.67)
+			(xy 844.55 83.82) (xy 844.55 201.93)
 		)
 		(stroke
@@
 	(wire
 		(pts
-			(xy 842.01 69.85) (xy 842.01 151.13)
-		)
-		(stroke
-			(width 0)
-			(type default)
-		)
-	)
-	(wire
-		(pts
 			(xy 62.23 530.86) (xy 74.93 530.86)
 		)
@@
 	(wire
 		(pts
-			(xy 595.63 148.59) (xy 839.47 148.59)
-		)
-		(stroke
-			(width 0)
-			(type default)
-		)
-	)
-	(wire
-		(pts
 			(xy 775.97 128.27) (xy 595.63 128.27)
 		)
@@
 	(wire
 		(pts
-			(xy 842.01 151.13) (xy 595.63 151.13)
-		)
-		(stroke
-			(width 0)
-			(type default)
-		)
-	)
-	(wire
-		(pts
 			(xy 29.21 530.86) (xy 29.21 520.7)
 		)
@@
 	(wire
 		(pts
-			(xy 847.09 99.06) (xy 847.09 156.21)
+			(xy 847.09 99.06) (xy 847.09 199.39)
 		)
 		(stroke
@@
 		)
 		(stroke
+			(width 0)
+			(type default)
+		)
+	)
+	(wire
+		(pts
+			(xy 842.01 69.85) (xy 842.01 204.47)
+		)
+		(stroke

Commit message: sync
Parts:
- F1: value 500mA -> 3A
Connections:
- net at LED411.3 (DOUT): now also LED390.1 (DIN)
- net at LED139.3 (DOUT): now also LED128.1 (DIN)
