File: Atrium PCB/Atrium PCB.kicad_pcb (KiCad board)
At the start: 2 copper layers, 415 parts, among them J1 Conn_01x05_Pin, SW1 EC11E09244BS, SW2 SKRPACE010, SW3 SKRPACE010, U12 AP2112K-3.3, U2 LSM6DS3TR-C, U6 SN74LVC1T45DBVR, X1 X322512MSB4SI

Commit message: sync
Parts:
- added D1: D, Diode_SMD:D_0603_1608Metric, F.Cu at (118.4, 150.8)
- added D11: D, Diode_SMD:D_0603_1608Metric, F.Cu at (122.5, 150.8)
- added D12: D, Diode_SMD:D_0603_1608Metric, F.Cu at (122.5, 153.4)
- added D13: D, Diode_SMD:D_0603_1608Metric, F.Cu at (122.5, 156.0)
- added D14: D, Diode_SMD:D_0603_1608Metric, F.Cu at (122.5, 158.5)
- added D16: D, Diode_SMD:D_0603_1608Metric, F.Cu at (122.5, 161.1)
- added D17: D, Diode_SMD:D_0603_1608Metric, F.Cu at (122.5, 163.7)
- added D18: D, Diode_SMD:D_0603_1608Metric, F.Cu at (122.5, 166.3)
- added D2: D, Diode_SMD:D_0603_1608Metric, F.Cu at (118.4, 153.4)
- added D20: D, Diode_SMD:D_0603_1608Metric, F.Cu at (126.5, 150.8)
- added D21: D, Diode_SMD:D_0603_1608Metric, F.Cu at (126.5, 153.4)
- added D22: D, Diode_SMD:D_0603_1608Metric, F.Cu at (126.5, 156.0)
- added D24: D, Diode_SMD:D_0603_1608Metric, F.Cu at (126.5, 158.5)
- added D25: D, Diode_SMD:D_0603_1608Metric, F.Cu at (126.5, 161.1)
- added D26: D, Diode_SMD:D_0603_1608Metric, F.Cu at (126.5, 163.7)
- added D28: D, Diode_SMD:D_0603_1608Metric, F.Cu at (126.5, 166.3)
- added D29: D, Diode_SMD:D_0603_1608Metric, F.Cu at (130.6, 150.8)
- added D3: D, Diode_SMD:D_0603_1608Metric, F.Cu at (118.4, 156.0)
- added D30: D, Diode_SMD:D_0603_1608Metric, F.Cu at (130.6, 153.4)
- added D32: D, Diode_SMD:D_0603_1608Metric, F.Cu at (130.6, 156.0)
- added D33: D, Diode_SMD:D_0603_1608Metric, F.Cu at (130.6, 158.5)
- added D34: D, Diode_SMD:D_0603_1608Metric, F.Cu at (130.6, 161.1)
- added D36: D, Diode_SMD:D_0603_1608Metric, F.Cu at (130.6, 163.7)
- added D37: D, Diode_SMD:D_0603_1608Metric, F.Cu at (130.6, 166.3)
- added D38: D, Diode_SMD:D_0603_1608Metric, F.Cu at (134.6, 150.8)
- added D40: D, Diode_SMD:D_0603_1608Metric, F.Cu at (134.6, 153.4)
- added D41: D, Diode_SMD:D_0603_1608Metric, F.Cu at (134.6, 156.0)
- added D42: D, Diode_SMD:D_0603_1608Metric, F.Cu at (134.6, 158.5)
- added D43: D, Diode_SMD:D_0603_1608Metric, F.Cu at (134.6, 161.1)
- added D44: D, Diode_SMD:D_0603_1608Metric, F.Cu at (134.6, 163.7)
- added D45: D, Diode_SMD:D_0603_1608Metric, F.Cu at (134.6, 166.3)
- added D46: D, Diode_SMD:D_0603_1608Metric, F.Cu at (138.7, 150.8)
- added D48: D, Diode_SMD:D_0603_1608Metric, F.Cu at (138.7, 153.4)
- added D49: D, Diode_SMD:D_0603_1608Metric, F.Cu at (138.7, 156.0)
- added D50: D, Diode_SMD:D_0603_1608Metric, F.Cu at (138.7, 158.5)
- added D51: D, Diode_SMD:D_0603_1608Metric, F.Cu at (138.7, 161.1)
- added D52: D, Diode_SMD:D_0603_1608Metric, F.Cu at (138.7, 163.7)
- added D6: D, Diode_SMD:D_0603_1608Metric, F.Cu at (118.4, 158.5)
- added D7: D, Diode_SMD:D_0603_1608Metric, F.Cu at (118.4, 161.1)
- added D8: D, Diode_SMD:D_0603_1608Metric, F.Cu at (118.4, 163.7)
- added D9: D, Diode_SMD:D_0603_1608Metric, F.Cu at (118.4, 166.3)
- added LED2: SK6805-EC15, easyeda2kicad:LED-SMD_4P-L1.5-W1.5-BL, F.Cu at (162.2, 189.3)
- added SW10: SW_Push, PCM_Switch_Keyboard_Hotswap_Kailh:SW_Hotswap_Kailh_Choc_V1V2_1.00u, F.Cu at (34.3, 29.1)
- added SW11: SW_Push, PCM_Switch_Keyboard_Hotswap_Kailh:SW_Hotswap_Kailh_Choc_V1V2_1.00u, F.Cu at (31.3, 46.1)
- added SW13: SW_Push, PCM_Switch_Keyboard_Hotswap_Kailh:SW_Hotswap_Kailh_Choc_V1V2_1.00u, F.Cu at (91.1, 77.7)
- added SW14: SW_Push, PCM_Switch_Keyboard_Hotswap_Kailh:SW_Hotswap_Kailh_Choc_V1V2_1.00u, F.Cu at (56.1, 11.4)
- added SW15: SW_Push, PCM_Switch_Keyboard_Hotswap_Kailh:SW_Hotswap_Kailh_Choc_V1V2_1.00u, F.Cu at (53.1, 28.3)
- added SW16: SW_Push, PCM_Switch_Keyboard_Hotswap_Kailh:SW_Hotswap_Kailh_Choc_V1V2_1.00u, F.Cu at (50.1, 45.3)
- added SW18: SW_Push, PCM_Switch_Keyboard_Hotswap_Kailh:SW_Hotswap_Kailh_Choc_V1V2_1.00u, F.Cu at (75.2, 10.6)
- added SW19: SW_Push, PCM_Switch_Keyboard_Hotswap_Kailh:SW_Hotswap_Kailh_Choc_V1V2_1.00u, F.Cu at (72.2, 27.6)
- added SW20: SW_Push, PCM_Switch_Keyboard_Hotswap_Kailh:SW_Hotswap_Kailh_Choc_V1V2_1.00u, F.Cu at (69.2, 44.5)
- added SW22: SW_Push, PCM_Switch_Keyboard_Hotswap_Kailh:SW_Hotswap_Kailh_Choc_V1V2_1.00u, F.Cu at (92.8, 17.9)
- added SW23: SW_Push, PCM_Switch_Keyboard_Hotswap_Kailh:SW_Hotswap_Kailh_Choc_V1V2_1.00u, F.Cu at (89.8, 34.9)
- added SW24: SW_Push, PCM_Switch_Keyboard_Hotswap_Kailh:SW_Hotswap_Kailh_Choc_V1V2_1.00u, F.Cu at (86.8, 51.9)
- added SW26: SW_Push, PCM_Switch_Keyboard_Hotswap_Kailh:SW_Hotswap_Kailh_Choc_V1V2_1.00u, F.Cu at (110.4, 25.0)
- added SW27: SW_Push, PCM_Switch_Keyboard_Hotswap_Kailh:SW_Hotswap_Kailh_Choc_V1V2_1.00u, F.Cu at (107.4, 42.0)
- added SW28: SW_Push, PCM_Switch_Keyboard_Hotswap_Kailh:SW_Hotswap_Kailh_Choc_V1V2_1.00u, F.Cu at (104.4, 59.0)
- added SW30: SW_Push, PCM_Switch_Keyboard_Hotswap_Kailh:SW_Hotswap_Kailh_Choc_V1V2_1.00u, F.Cu at (138.0, 25.0)
- added SW31: SW_Push, PCM_Switch_Keyboard_Hotswap_Kailh:SW_Hotswap_Kailh_Choc_V1V2_1.00u, F.Cu at (141.0, 42.0)
- added SW32: SW_Push, PCM_Switch_Keyboard_Hotswap_Kailh:SW_Hotswap_Kailh_Choc_V1V2_1.00u, F.Cu at (144.0, 59.0)
- added SW34: SW_Push, PCM_Switch_Keyboard_Hotswap_Kailh:SW_Hotswap_Kailh_Choc_V1V2_1.00u, F.Cu at (155.7, 17.8)
- added SW35: SW_Push, PCM_Switch_Keyboard_Hotswap_Kailh:SW_Hotswap_Kailh_Choc_V1V2_1.00u, F.Cu at (158.7, 34.7)
- added SW36: SW_Push, PCM_Switch_Keyboard_Hotswap_Kailh:SW_Hotswap_Kailh_Choc_V1V2_1.00u, F.Cu at (161.7, 51.7)
- added SW38: SW_Push, PCM_Switch_Keyboard_Hotswap_Kailh:SW_Hotswap_Kailh_Choc_V1V2_1.00u, F.Cu at (173.1, 10.6)
- added SW39: SW_Push, PCM_Switch_Keyboard_Hotswap_Kailh:SW_Hotswap_Kailh_Choc_V1V2_1.00u, F.Cu at (176.1, 27.6)
- added SW4: SW_Push, PCM_Switch_Keyboard_Hotswap_Kailh:SW_Hotswap_Kailh_Choc_V1V2_1.00u, F.Cu at (17.9, 12.9)
- added SW40: SW_Push, PCM_Switch_Keyboard_Hotswap_Kailh:SW_Hotswap_Kailh_Choc_V1V2_1.00u, F.Cu at (179.1, 44.6)
- added SW42: SW_Push, PCM_Switch_Keyboard_Hotswap_Kailh:SW_Hotswap_Kailh_Choc_V1V2_1.00u, F.Cu at (192.1, 11.4)
- added SW43: SW_Push, PCM_Switch_Keyboard_Hotswap_Kailh:SW_Hotswap_Kailh_Choc_V1V2_1.00u, F.Cu at (195.1, 28.4)
- added SW44: SW_Push, PCM_Switch_Keyboard_Hotswap_Kailh:SW_Hotswap_Kailh_Choc_V1V2_1.00u, F.Cu at (198.1, 45.4)
- added SW45: SW_Push, PCM_Switch_Keyboard_Hotswap_Kailh:SW_Hotswap_Kailh_Choc_V1V2_1.00u, F.Cu at (211.1, 12.1)
- added SW46: SW_Push, PCM_Switch_Keyboard_Hotswap_Kailh:SW_Hotswap_Kailh_Choc_V1V2_1.00u, F.Cu at (72.8, 74.5)
- added SW47: SW_Push, PCM_Switch_Keyboard_Hotswap_Kailh:SW_Hotswap_Kailh_Choc_V1V2_1.00u, F.Cu at (157.5, 78.2)
- added SW48: SW_Push, PCM_Switch_Keyboard_Hotswap_Kailh:SW_Hotswap_Kailh_Choc_V1V2_1.00u, F.Cu at (176.8, 74.8)
- added SW5: SW_Push, PCM_Switch_Keyboard_Hotswap_Kailh:SW_Hotswap_Kailh_Choc_V1V2_1.00u, F.Cu at (14.9, 29.9)
- added SW50: SW_Push, PCM_Switch_Keyboard_Hotswap_Kailh:SW_Hotswap_Kailh_Choc_V1V2_1.00u, F.Cu at (214.1, 29.0)
- added SW51: SW_Push, PCM_Switch_Keyboard_Hotswap_Kailh:SW_Hotswap_Kailh_Choc_V1V2_1.00u, F.Cu at (217.1, 46.0)
- added SW52: SW_Push, PCM_Switch_Keyboard_Hotswap_Kailh:SW_Hotswap_Kailh_Choc_V1V2_1.00u, F.Cu at (230.0, 13.0)
- added SW53: SW_Push, PCM_Switch_Keyboard_Hotswap_Kailh:SW_Hotswap_Kailh_Choc_V1V2_1.00u, F.Cu at (233.0, 30.0)
- added SW54: SW_Push, PCM_Switch_Keyboard_Hotswap_Kailh:SW_Hotswap_Kailh_Choc_V1V2_1.00u, F.Cu at (236.0, 47.0)
- added SW6: SW_Push, PCM_Switch_Keyboard_Hotswap_Kailh:SW_Hotswap_Kailh_Choc_V1V2_1.00u, F.Cu at (11.9, 46.9)
- added SW8: SW_Push, PCM_Switch_Keyboard_Hotswap_Kailh:SW_Hotswap_Kailh_Choc_V1V2_2.00u, F.Cu at (123.6, 80.6)
- added SW9: SW_Push, PCM_Switch_Keyboard_Hotswap_Kailh:SW_Hotswap_Kailh_Choc_V1V2_1.00u, F.Cu at (37.3, 12.1)
- moved SW1 155.1 mm to (242.5, 65.7), turned to 10 degrees
- moved LED176 155.0 mm to (29.2, 164.3)
- moved LED177 155.0 mm to (29.2, 168.9)
- moved D5 134.8 mm to (138.1, 188.4)
- moved R40 134.5 mm to (162.0, 184.8)
- moved R41 134.5 mm to (162.0, 186.8)
- moved J1 132.9 mm to (143.9, 177.1)
- moved FB1 132.1 mm to (126.3, 186.4)
- moved TP18 129.2 mm to (160.2, 151.3)
- moved TP19 129.2 mm to (160.2, 154.8)
- moved TP21 129.2 mm to (160.2, 161.9)
- moved TP22 129.2 mm to (160.2, 165.5)
- moved TP20 129.2 mm to (160.2, 158.4)
- moved FPC1 124.1 mm to (212.8, 119.2), turned to 180 degrees
- moved U12 122.5 mm to (148.8, 185.9)
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Other:
- board outline added: 256.3 x 95.5 mm

Commit message: sync
Parts:
- removed C202, C203, C204, C205, C206, C207, C208, C209, C210, C212, C213, C214, C215, C216, C217, C218, C219, C220, C221, C49, C50, C51, C52, C53, C54, C55, C56, C57, C58, C59, C60, C61, C66, C67, C68, C69, C70, C71, C72, C73, C74, C75, C76, C77, C78, C79, C80, C81: 100nF, Capacitor_SMD:C_0603_1608Metric
- removed D1, D11, D12, D13, D14, D16, D17, D18, D2, D20, D21, D22, D24, D25, D26, D28, D29, D3, D30, D32, D33, D34, D36, D37, D38, D40, D41, D42, D43, D44, D45, D46, D48, D49, D50, D51, D52, D6, D7, D8, D9: D, Diode_SMD:D_0603_1608Metric
- removed LED175, LED176, LED177, LED178, LED179, LED180, LED181, LED182, LED183, LED184, LED185, LED186, LED187, LED188, LED189, LED190, LED191, LED192, LED193, LED194, LED195, LED196, LED197, LED198, LED199, LED200, LED201, LED202, LED203, LED204, LED205, LED206, LED207, LED208, LED209, LED210, LED211, LED212, LED213, LED214, LED215, LED216, LED217, LED218, LED219, LED220, LED221, LED222, LED223, LED224, LED225, LED226, LED227, LED228, LED229, LED230, LED231, LED232, LED233, LED234, LED235, LED236, LED237, LED238, LED239, LED240, LED241, LED242, LED243, LED244, LED245, LED246, LED247, LED248, LED249, LED250, LED251, LED252, LED253, LED254, LED255, LED256, LED257, LED258, LED259, LED260, LED261, LED262, LED263, LED264, LED265, LED266, LED267, LED268, LED269, LED270, LED271, LED272, LED273, LED274, LED275, LED276, LED277, LED278, LED279, LED280, LED281, LED282, LED283, LED284, LED285, LED286, LED287, LED288, LED289, LED290, LED291, LED292, LED293, LED294, LED295, LED296, LED297, LED298, LED299, LED300, LED301, LED302, LED303, LED304, LED305, LED306, LED307, LED308, LED309, LED310, LED311, LED312, LED313, LED314, LED315, LED316, LED317, LED318, LED319, LED320, LED321, LED322, LED323, LED324, LED325, LED326, LED327, LED328, LED329, LED330, LED331, LED332, LED333, LED334, LED335, LED336, LED337, LED338, LED339, LED340, LED341, LED342, STATUS1: SK6812MINI-E_C5149201, easyeda2kicad:LED-SMD_4P-L3.2-W2.8-LS5.9_SK6812MINI-E
- removed R11, R12, R14, R15, R16: 470, Resistor_SMD:R_0603_1608Metric
- added C383: 100nF, Capacitor_SMD:C_0402_1005Metric, F.Cu at (274.2, 120.8)
- added C384: 100nF, Capacitor_SMD:C_0402_1005Metric, F.Cu at (274.2, 122.8)
- added C385: 100nF, Capacitor_SMD:C_0402_1005Metric, F.Cu at (274.2, 124.8)
- added C386: 100nF, Capacitor_SMD:C_0402_1005Metric, F.Cu at (274.2, 126.7)
- added C387: 100nF, Capacitor_SMD:C_0402_1005Metric, F.Cu at (274.2, 128.7)
- added C388: 100nF, Capacitor_SMD:C_0402_1005Metric, F.Cu at (274.2, 130.7)
- added C389: 100nF, Capacitor_SMD:C_0402_1005Metric, F.Cu at (274.2, 132.7)
- added C390: 100nF, Capacitor_SMD:C_0402_1005Metric, F.Cu at (274.2, 134.6)
- added C391: 100nF, Capacitor_SMD:C_0402_1005Metric, F.Cu at (274.2, 136.6)
- added C392: 100nF, Capacitor_SMD:C_0402_1005Metric, F.Cu at (277.0, 120.8)
- added C393: 100nF, Capacitor_SMD:C_0402_1005Metric, F.Cu at (277.0, 122.8)
- added C394: 100nF, Capacitor_SMD:C_0402_1005Metric, F.Cu at (277.0, 124.8)
- added C395: 100nF, Capacitor_SMD:C_0402_1005Metric, F.Cu at (277.0, 126.7)
- added C396: 100nF, Capacitor_SMD:C_0402_1005Metric, F.Cu at (277.0, 128.7)
- added C397: 100nF, Capacitor_SMD:C_0402_1005Metric, F.Cu at (277.0, 130.7)
- added C398: 100nF, Capacitor_SMD:C_0402_1005Metric, F.Cu at (277.0, 132.7)
- added C399: 100nF, Capacitor_SMD:C_0402_1005Metric, F.Cu at (277.0, 134.6)
- added C402: 100nF, Capacitor_SMD:C_0402_1005Metric, F.Cu at (277.0, 136.6)
- added C403: 100nF, Capacitor_SMD:C_0402_1005Metric, F.Cu at (279.9, 120.8)
- added C404: 100nF, Capacitor_SMD:C_0402_1005Metric, F.Cu at (279.9, 122.8)
- added C405: 100nF, Capacitor_SMD:C_0402_1005Metric, F.Cu at (279.9, 124.8)
- added C406: 100nF, Capacitor_SMD:C_0402_1005Metric, F.Cu at (279.9, 126.7)
- added C407: 100nF, Capacitor_SMD:C_0402_1005Metric, F.Cu at (279.9, 128.7)
- added C408: 100nF, Capacitor_SMD:C_0402_1005Metric, F.Cu at (279.9, 130.7)
- added C409: 100nF, Capacitor_SMD:C_0402_1005Metric, F.Cu at (279.9, 132.7)
- added C410: 100nF, Capacitor_SMD:C_0402_1005Metric, F.Cu at (279.9, 134.6)
- added C411: 100nF, Capacitor_SMD:C_0402_1005Metric, F.Cu at (279.9, 136.6)
- added C412: 100nF, Capacitor_SMD:C_0402_1005Metric, F.Cu at (282.8, 120.8)
- added C413: 100nF, Capacitor_SMD:C_0402_1005Metric, F.Cu at (282.8, 122.8)
- added C414: 100nF, Capacitor_SMD:C_0402_1005Metric, F.Cu at (282.8, 124.8)
- added C415: 100nF, Capacitor_SMD:C_0402_1005Metric, F.Cu at (282.8, 126.7)
- added C416: 100nF, Capacitor_SMD:C_0402_1005Metric, F.Cu at (282.8, 128.7)
- added C417: 100nF, Capacitor_SMD:C_0402_1005Metric, F.Cu at (282.8, 130.7)
- added C418: 100nF, Capacitor_SMD:C_0402_1005Metric, F.Cu at (282.8, 132.7)
- added C419: 100nF, Capacitor_SMD:C_0402_1005Metric, F.Cu at (282.8, 134.6)
- added C420: 100nF, Capacitor_SMD:C_0402_1005Metric, F.Cu at (282.8, 136.6)
- added C421: 100nF, Capacitor_SMD:C_0402_1005Metric, F.Cu at (285.6, 120.8)
- added C422: 100nF, Capacitor_SMD:C_0402_1005Metric, F.Cu at (285.6, 122.8)
- added C423: 100nF, Capacitor_SMD:C_0402_1005Metric, F.Cu at (285.6, 124.8)
- added C424: 100nF, Capacitor_SMD:C_0402_1005Metric, F.Cu at (285.6, 126.7)
- added J2: Conn_01x05_Pin, Connector_PinHeader_2.54mm:PinHeader_1x05_P2.54mm_Vertical, F.Cu at (41.4, 86.1)
- added J3: Conn_01x04_Pin, Connector_PinHeader_2.54mm:PinHeader_1x04_P2.54mm_Vertical, F.Cu at (34.5, 81.2)
- added LED10: SK6805-EC15, easyeda2kicad:LED-SMD_4P-L1.5-W1.5-BL, F.Cu at (7.64, 20.0)
- added LED100: SK6805-EC15, easyeda2kicad:LED-SMD_4P-L1.5-W1.5-BL, F.Cu at (261.1, 176.5)
- added LED101: SK6805-EC15, easyeda2kicad:LED-SMD_4P-L1.5-W1.5-BL, F.Cu at (261.1, 179.6)
- added LED102: SK6805-EC15, easyeda2kicad:LED-SMD_4P-L1.5-W1.5-BL, F.Cu at (261.1, 182.7)
- added LED103: SK6805-EC15, easyeda2kicad:LED-SMD_4P-L1.5-W1.5-BL, F.Cu at (264.2, 151.4)
- added LED104: SK6805-EC15, easyeda2kicad:LED-SMD_4P-L1.5-W1.5-BL, F.Cu at (264.2, 154.6)
- added LED105: SK6805-EC15, easyeda2kicad:LED-SMD_4P-L1.5-W1.5-BL, F.Cu at (264.2, 157.7)
- added LED106: SK6805-EC15, easyeda2kicad:LED-SMD_4P-L1.5-W1.5-BL, F.Cu at (264.2, 160.8)
- added LED107: SK6805-EC15, easyeda2kicad:LED-SMD_4P-L1.5-W1.5-BL, F.Cu at (264.2, 163.9)
- added LED108: SK6805-EC15, easyeda2kicad:LED-SMD_4P-L1.5-W1.5-BL, F.Cu at (264.2, 167.1)
- added LED109: SK6805-EC15, easyeda2kicad:LED-SMD_4P-L1.5-W1.5-BL, F.Cu at (264.2, 170.2)
- added LED11: SK6805-EC15, easyeda2kicad:LED-SMD_4P-L1.5-W1.5-BL, F.Cu at (-39.2, 101.4)
- added LED110: SK6805-EC15, easyeda2kicad:LED-SMD_4P-L1.5-W1.5-BL, F.Cu at (264.2, 173.3)
- added LED111: SK6805-EC15, easyeda2kicad:LED-SMD_4P-L1.5-W1.5-BL, F.Cu at (264.2, 176.5)
- added LED112: SK6805-EC15, easyeda2kicad:LED-SMD_4P-L1.5-W1.5-BL, F.Cu at (264.2, 179.6)
- added LED113: SK6805-EC15, easyeda2kicad:LED-SMD_4P-L1.5-W1.5-BL, F.Cu at (264.2, 182.7)
- added LED114: SK6805-EC15, easyeda2kicad:LED-SMD_4P-L1.5-W1.5-BL, F.Cu at (267.3, 151.4)
- added LED115: SK6805-EC15, easyeda2kicad:LED-SMD_4P-L1.5-W1.5-BL, F.Cu at (267.3, 154.6)
- added LED116: SK6805-EC15, easyeda2kicad:LED-SMD_4P-L1.5-W1.5-BL, F.Cu at (267.3, 157.7)
- added LED117: SK6805-EC15, easyeda2kicad:LED-SMD_4P-L1.5-W1.5-BL, F.Cu at (267.3, 160.8)
- added LED118: SK6805-EC15, easyeda2kicad:LED-SMD_4P-L1.5-W1.5-BL, F.Cu at (267.3, 163.9)
- added LED119: SK6805-EC15, easyeda2kicad:LED-SMD_4P-L1.5-W1.5-BL, F.Cu at (267.3, 167.1)
- added LED12: SK6805-EC15, easyeda2kicad:LED-SMD_4P-L1.5-W1.5-BL, F.Cu at (-39.2, 104.5)
- added LED120: SK6805-EC15, easyeda2kicad:LED-SMD_4P-L1.5-W1.5-BL, F.Cu at (267.3, 170.2)
- added LED121: SK6805-EC15, easyeda2kicad:LED-SMD_4P-L1.5-W1.5-BL, F.Cu at (267.3, 173.3)
- added LED122: SK6805-EC15, easyeda2kicad:LED-SMD_4P-L1.5-W1.5-BL, F.Cu at (171.6, 152.6)
- added LED13: SK6805-EC15, easyeda2kicad:LED-SMD_4P-L1.5-W1.5-BL, F.Cu at (-39.2, 107.6)
- added LED14: SK6805-EC15, easyeda2kicad:LED-SMD_4P-L1.5-W1.5-BL, F.Cu at (-39.2, 110.8)
- added LED15: SK6805-EC15, easyeda2kicad:LED-SMD_4P-L1.5-W1.5-BL, F.Cu at (-39.2, 113.9)
- added LED16: SK6805-EC15, easyeda2kicad:LED-SMD_4P-L1.5-W1.5-BL, F.Cu at (-39.2, 117.0)
- added LED17: SK6805-EC15, easyeda2kicad:LED-SMD_4P-L1.5-W1.5-BL, F.Cu at (28.7, 6.14)
- added LED18: SK6805-EC15, easyeda2kicad:LED-SMD_4P-L1.5-W1.5-BL, F.Cu at (-36.1, 101.4)
- added LED19: SK6805-EC15, easyeda2kicad:LED-SMD_4P-L1.5-W1.5-BL, F.Cu at (-36.1, 104.5)
- added LED20: SK6805-EC15, easyeda2kicad:LED-SMD_4P-L1.5-W1.5-BL, F.Cu at (-36.1, 107.6)
- added LED21: SK6805-EC15, easyeda2kicad:LED-SMD_4P-L1.5-W1.5-BL, F.Cu at (-36.1, 110.8)
- added LED22: SK6805-EC15, easyeda2kicad:LED-SMD_4P-L1.5-W1.5-BL, F.Cu at (-36.1, 113.9)
- added LED23: SK6805-EC15, easyeda2kicad:LED-SMD_4P-L1.5-W1.5-BL, F.Cu at (242.3, 151.4)
- added LED24: SK6805-EC15, easyeda2kicad:LED-SMD_4P-L1.5-W1.5-BL, F.Cu at (25.6, 23.1)
- added LED25: SK6805-EC15, easyeda2kicad:LED-SMD_4P-L1.5-W1.5-BL, F.Cu at (242.3, 154.6)
- added LED26: SK6805-EC15, easyeda2kicad:LED-SMD_4P-L1.5-W1.5-BL, F.Cu at (-33.0, 104.5)
- added LED27: SK6805-EC15, easyeda2kicad:LED-SMD_4P-L1.5-W1.5-BL, F.Cu at (242.3, 157.7)
- added LED28: SK6805-EC15, easyeda2kicad:LED-SMD_4P-L1.5-W1.5-BL, F.Cu at (-33.0, 110.8)
- added LED29: SK6805-EC15, easyeda2kicad:LED-SMD_4P-L1.5-W1.5-BL, F.Cu at (242.3, 160.8)
- added LED3: SK6805-EC15, easyeda2kicad:LED-SMD_4P-L1.5-W1.5-BL, F.Cu at (10.9, 2.90)
- added LED30: SK6805-EC15, easyeda2kicad:LED-SMD_4P-L1.5-W1.5-BL, F.Cu at (242.3, 163.9)
- added LED31: SK6805-EC15, easyeda2kicad:LED-SMD_4P-L1.5-W1.5-BL, F.Cu at (242.3, 167.1)
- added LED32: SK6805-EC15, easyeda2kicad:LED-SMD_4P-L1.5-W1.5-BL, F.Cu at (242.3, 170.2)
- added LED33: SK6805-EC15, easyeda2kicad:LED-SMD_4P-L1.5-W1.5-BL, F.Cu at (242.3, 173.3)
- added LED34: SK6805-EC15, easyeda2kicad:LED-SMD_4P-L1.5-W1.5-BL, F.Cu at (242.3, 176.5)
- added LED35: SK6805-EC15, easyeda2kicad:LED-SMD_4P-L1.5-W1.5-BL, F.Cu at (242.3, 179.6)
- added LED36: SK6805-EC15, easyeda2kicad:LED-SMD_4P-L1.5-W1.5-BL, F.Cu at (242.3, 182.7)
- added LED37: SK6805-EC15, easyeda2kicad:LED-SMD_4P-L1.5-W1.5-BL, F.Cu at (245.4, 151.4)
- added LED38: SK6805-EC15, easyeda2kicad:LED-SMD_4P-L1.5-W1.5-BL, F.Cu at (245.4, 154.6)
- added LED39: SK6805-EC15, easyeda2kicad:LED-SMD_4P-L1.5-W1.5-BL, F.Cu at (245.4, 157.7)
- added LED4: SK6805-EC15, easyeda2kicad:LED-SMD_4P-L1.5-W1.5-BL, F.Cu at (4.55, 37.0)
- added LED40: SK6805-EC15, easyeda2kicad:LED-SMD_4P-L1.5-W1.5-BL, F.Cu at (245.4, 160.8)
- added LED41: SK6805-EC15, easyeda2kicad:LED-SMD_4P-L1.5-W1.5-BL, F.Cu at (245.4, 163.9)
- added LED42: SK6805-EC15, easyeda2kicad:LED-SMD_4P-L1.5-W1.5-BL, F.Cu at (245.4, 167.1)
- added LED43: SK6805-EC15, easyeda2kicad:LED-SMD_4P-L1.5-W1.5-BL, F.Cu at (245.4, 170.2)
- added LED44: SK6805-EC15, easyeda2kicad:LED-SMD_4P-L1.5-W1.5-BL, F.Cu at (245.4, 173.3)
- added LED45: SK6805-EC15, easyeda2kicad:LED-SMD_4P-L1.5-W1.5-BL, F.Cu at (245.4, 176.5)
- added LED46: SK6805-EC15, easyeda2kicad:LED-SMD_4P-L1.5-W1.5-BL, F.Cu at (245.4, 179.6)
- added LED47: SK6805-EC15, easyeda2kicad:LED-SMD_4P-L1.5-W1.5-BL, F.Cu at (245.4, 182.7)
- added LED48: SK6805-EC15, easyeda2kicad:LED-SMD_4P-L1.5-W1.5-BL, F.Cu at (248.6, 151.4)
- added LED49: SK6805-EC15, easyeda2kicad:LED-SMD_4P-L1.5-W1.5-BL, F.Cu at (248.6, 154.6)
- added LED5: SK6805-EC15, easyeda2kicad:LED-SMD_4P-L1.5-W1.5-BL, F.Cu at (-42.4, 104.5)
- added LED50: SK6805-EC15, easyeda2kicad:LED-SMD_4P-L1.5-W1.5-BL, F.Cu at (248.6, 157.7)
- added LED51: SK6805-EC15, easyeda2kicad:LED-SMD_4P-L1.5-W1.5-BL, F.Cu at (248.6, 160.8)
- added LED52: SK6805-EC15, easyeda2kicad:LED-SMD_4P-L1.5-W1.5-BL, F.Cu at (248.6, 163.9)
- added LED53: SK6805-EC15, easyeda2kicad:LED-SMD_4P-L1.5-W1.5-BL, F.Cu at (248.6, 167.1)
- added LED54: SK6805-EC15, easyeda2kicad:LED-SMD_4P-L1.5-W1.5-BL, F.Cu at (248.6, 170.2)
- added LED55: SK6805-EC15, easyeda2kicad:LED-SMD_4P-L1.5-W1.5-BL, F.Cu at (248.6, 173.3)
- added LED56: SK6805-EC15, easyeda2kicad:LED-SMD_4P-L1.5-W1.5-BL, F.Cu at (248.6, 176.5)
- added LED57: SK6805-EC15, easyeda2kicad:LED-SMD_4P-L1.5-W1.5-BL, F.Cu at (248.6, 179.6)
- added LED58: SK6805-EC15, easyeda2kicad:LED-SMD_4P-L1.5-W1.5-BL, F.Cu at (248.6, 182.7)
- added LED59: SK6805-EC15, easyeda2kicad:LED-SMD_4P-L1.5-W1.5-BL, F.Cu at (251.7, 151.4)
- added LED6: SK6805-EC15, easyeda2kicad:LED-SMD_4P-L1.5-W1.5-BL, F.Cu at (-42.4, 107.6)
- added LED60: SK6805-EC15, easyeda2kicad:LED-SMD_4P-L1.5-W1.5-BL, F.Cu at (251.7, 154.6)
- added LED61: SK6805-EC15, easyeda2kicad:LED-SMD_4P-L1.5-W1.5-BL, F.Cu at (251.7, 157.7)
- added LED62: SK6805-EC15, easyeda2kicad:LED-SMD_4P-L1.5-W1.5-BL, F.Cu at (251.7, 160.8)
- added LED63: SK6805-EC15, easyeda2kicad:LED-SMD_4P-L1.5-W1.5-BL, F.Cu at (251.7, 163.9)
- added LED64: SK6805-EC15, easyeda2kicad:LED-SMD_4P-L1.5-W1.5-BL, F.Cu at (251.7, 167.1)
- added LED65: SK6805-EC15, easyeda2kicad:LED-SMD_4P-L1.5-W1.5-BL, F.Cu at (251.7, 170.2)
- added LED66: SK6805-EC15, easyeda2kicad:LED-SMD_4P-L1.5-W1.5-BL, F.Cu at (251.7, 173.3)
- added LED67: SK6805-EC15, easyeda2kicad:LED-SMD_4P-L1.5-W1.5-BL, F.Cu at (251.7, 176.5)
- added LED68: SK6805-EC15, easyeda2kicad:LED-SMD_4P-L1.5-W1.5-BL, F.Cu at (251.7, 179.6)
- added LED69: SK6805-EC15, easyeda2kicad:LED-SMD_4P-L1.5-W1.5-BL, F.Cu at (251.7, 182.7)
- added LED7: SK6805-EC15, easyeda2kicad:LED-SMD_4P-L1.5-W1.5-BL, F.Cu at (-42.4, 110.8)
- added LED70: SK6805-EC15, easyeda2kicad:LED-SMD_4P-L1.5-W1.5-BL, F.Cu at (254.8, 151.4)
- added LED71: SK6805-EC15, easyeda2kicad:LED-SMD_4P-L1.5-W1.5-BL, F.Cu at (254.8, 154.6)
- added LED72: SK6805-EC15, easyeda2kicad:LED-SMD_4P-L1.5-W1.5-BL, F.Cu at (254.8, 157.7)
- added LED73: SK6805-EC15, easyeda2kicad:LED-SMD_4P-L1.5-W1.5-BL, F.Cu at (254.8, 160.8)
- added LED74: SK6805-EC15, easyeda2kicad:LED-SMD_4P-L1.5-W1.5-BL, F.Cu at (254.8, 163.9)
- added LED75: SK6805-EC15, easyeda2kicad:LED-SMD_4P-L1.5-W1.5-BL, F.Cu at (254.8, 167.1)
- added LED76: SK6805-EC15, easyeda2kicad:LED-SMD_4P-L1.5-W1.5-BL, F.Cu at (254.8, 170.2)
- added LED77: SK6805-EC15, easyeda2kicad:LED-SMD_4P-L1.5-W1.5-BL, F.Cu at (254.8, 173.3)
- added LED78: SK6805-EC15, easyeda2kicad:LED-SMD_4P-L1.5-W1.5-BL, F.Cu at (254.8, 176.5)
- added LED79: SK6805-EC15, easyeda2kicad:LED-SMD_4P-L1.5-W1.5-BL, F.Cu at (254.8, 179.6)
- added LED8: SK6805-EC15, easyeda2kicad:LED-SMD_4P-L1.5-W1.5-BL, F.Cu at (-42.4, 113.9)
- added LED80: SK6805-EC15, easyeda2kicad:LED-SMD_4P-L1.5-W1.5-BL, F.Cu at (254.8, 182.7)
- added LED81: SK6805-EC15, easyeda2kicad:LED-SMD_4P-L1.5-W1.5-BL, F.Cu at (258.0, 151.4)
- added LED82: SK6805-EC15, easyeda2kicad:LED-SMD_4P-L1.5-W1.5-BL, F.Cu at (258.0, 154.6)
- added LED83: SK6805-EC15, easyeda2kicad:LED-SMD_4P-L1.5-W1.5-BL, F.Cu at (258.0, 157.7)
- added LED84: SK6805-EC15, easyeda2kicad:LED-SMD_4P-L1.5-W1.5-BL, F.Cu at (258.0, 160.8)
- added LED85: SK6805-EC15, easyeda2kicad:LED-SMD_4P-L1.5-W1.5-BL, F.Cu at (258.0, 163.9)
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Connections:
- LED2 pad 1: unconnected-(LED2-DIN-Pad1) -> Net-(LED2-DIN)
- LED2 pad 2: unconnected-(LED2-VDD-Pad2) -> +5V_LED
- LED2 pad 3: unconnected-(LED2-DOUT-Pad3) -> Net-(LED2-DOUT)
- LED2 pad 4: unconnected-(LED2-GND-Pad4) -> GND
- R13 pad 1: Net-(LED236-DIN) -> Net-(LED2-DIN)
- RP2350 pad 10: COL_8 -> Net-(J2-Pin_5)
- RP2350 pad 12: COL_9 -> Net-(J2-Pin_4)
- RP2350 pad 13: COL_10 -> Net-(J2-Pin_3)
- RP2350 pad 14: COL_11 -> Net-(J2-Pin_2)
- RP2350 pad 15: COL_12 -> Net-(J2-Pin_1)
- RP2350 pad 16: ROW_1 -> Net-(J3-Pin_4)
- RP2350 pad 17: ROW_2 -> Net-(J3-Pin_3)
- RP2350 pad 18: ROW_3 -> Net-(J3-Pin_2)
- RP2350 pad 19: ROW_4 -> Net-(J3-Pin_1)
- RP2350 pad 2: COL_1 -> MUX_S0
- RP2350 pad 3: COL_2 -> MUX_S1
- RP2350 pad 4: COL_3 -> MUX_S2
- RP2350 pad 40: ENC_A -> MUX_1
- RP2350 pad 41: ENC_B -> MUX_2
- RP2350 pad 42: ENC_SW -> MUX_3
- RP2350 pad 5: COL_4 -> MUX_S3
- RP2350 pad 7: COL_5 -> ENC_A
- RP2350 pad 8: COL_6 -> ENC_B
- RP2350 pad 9: COL_7 -> ENC_SW
Other:
- board size 256.3 x 95.5 mm -> 250.3 x 101.3 mm

Commit message: sync
Parts:
- moved FPC1 218.5 mm to (245.1, 25.6), turned to 90 degrees
- moved F1 189.8 mm to (17.3, 59.0)
- moved C400 180.2 mm to (21.1, 61.3), turned to 180 degrees
- moved U12 177.1 mm to (25.0, 59.2)
- moved C401 176.1 mm to (28.8, 61.1), turned to 90 degrees
- moved LED1 175.7 mm to (247.3, 35.9), turned to -90 degrees
- moved R40 173.0 mm to (245.6, 33.3), turned to -90 degrees
- moved R32 171.8 mm to (8.03, 55.5), turned to 90 degrees
- moved R33 170.2 mm to (8.10, 61.6), turned to 90 degrees
- moved R41 170.1 mm to (245.6, 38.7), turned to 90 degrees
- moved U6 162.2 mm to (33.7, 60.2)
- moved FB1 160.3 mm to (25.0, 62.1)
- moved C301 156.6 mm to (30.7, 61.1), turned to 90 degrees
- moved C382 156.5 mm to (30.7, 63.2), turned to -90 degrees
- moved C211 152.7 mm to (31.7, 63.2), turned to 90 degrees
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
Commit message: sync
Parts:
- removed C121, C157, C190: 100nF, Capacitor_SMD:C_0603_1608Metric
- removed FPC1: FPC-05F-12PH20, easyeda2kicad:FPC-SMD_12P-P0.50_FPC-05F-12PH20
- removed J2: Conn_01x05_Pin, Connector_PinHeader_2.54mm:PinHeader_1x05_P2.54mm_Vertical
- removed J3: Conn_01x04_Pin, Connector_PinHeader_2.54mm:PinHeader_1x04_P2.54mm_Vertical
- removed LED122, LED54, LED86: SK6805-EC15, easyeda2kicad:LED-SMD_4P-L1.5-W1.5-BL
- removed SW1: EC11E09244BS, easyeda2kicad:SW-TH_EC11XXXXXXXX
- removed SW10, SW11, SW13, SW14, SW15, SW16, SW18, SW19, SW20, SW22, SW23, SW24, SW26, SW27, SW28, SW30, SW31, SW32, SW34, SW35, SW36, SW38, SW39, SW4, SW40, SW42, SW43, SW44, SW45, SW46, SW47, SW48, SW5, SW50, SW51, SW52, SW53, SW54, SW6, SW8, SW9: SW_Push, PCM_Switch_Keyboard_Cherry_MX:SW_Cherry_MX_PCB
- added C202: 100nF, Capacitor_SMD:C_0603_1608Metric, F.Cu at (183.2, 20.5)
- added C203: 100nF, Capacitor_SMD:C_0603_1608Metric, F.Cu at (177.2, 20.5)
- added C204: 100nF, Capacitor_SMD:C_0603_1608Metric, F.Cu at (171.2, 20.5)
- added C205: 100nF, Capacitor_SMD:C_0603_1608Metric, F.Cu at (165.2, 20.5)
- added C206: 100nF, Capacitor_SMD:C_0603_1608Metric, F.Cu at (153.2, 20.5)
- added C207: 100nF, Capacitor_SMD:C_0603_1608Metric, F.Cu at (147.2, 20.5)
- added C208: 100nF, Capacitor_SMD:C_0603_1608Metric, F.Cu at (135.2, 20.5)
- added C209: 100nF, Capacitor_SMD:C_0603_1608Metric, F.Cu at (129.2, 20.5)
- added C210: 100nF, Capacitor_SMD:C_0603_1608Metric, F.Cu at (123.2, 20.5)
- added C212: 100nF, Capacitor_SMD:C_0603_1608Metric, F.Cu at (111.2, 20.5)
- added C213: 100nF, Capacitor_SMD:C_0603_1608Metric, F.Cu at (105.2, 20.5)
- added C214: 100nF, Capacitor_SMD:C_0603_1608Metric, F.Cu at (93.2, 20.5)
- added C215: 100nF, Capacitor_SMD:C_0603_1608Metric, F.Cu at (87.2, 20.5)
- added C216: 100nF, Capacitor_SMD:C_0603_1608Metric, F.Cu at (81.2, 20.5)
- added C217: 100nF, Capacitor_SMD:C_0603_1608Metric, F.Cu at (75.2, 20.5)
- added C218: 100nF, Capacitor_SMD:C_0603_1608Metric, F.Cu at (69.2, 20.5)
- added C219: 100nF, Capacitor_SMD:C_0603_1608Metric, F.Cu at (63.2, 20.5)
- added C220: 100nF, Capacitor_SMD:C_0603_1608Metric, F.Cu at (57.2, 20.5)
- added C221: 100nF, Capacitor_SMD:C_0603_1608Metric, F.Cu at (51.2, 20.5)
- added C222: 100nF, Capacitor_SMD:C_0603_1608Metric, F.Cu at (45.2, 20.5)
- added C223: 100nF, Capacitor_SMD:C_0603_1608Metric, F.Cu at (39.2, 20.5)
- added C224: 100nF, Capacitor_SMD:C_0603_1608Metric, F.Cu at (33.2, 20.5)
- added C225: 100nF, Capacitor_SMD:C_0603_1608Metric, F.Cu at (27.2, 20.5)
- added C226: 100nF, Capacitor_SMD:C_0603_1608Metric, F.Cu at (21.2, 20.5)
- added C227: 100nF, Capacitor_SMD:C_0603_1608Metric, F.Cu at (15.2, 20.5)
- added C228: 100nF, Capacitor_SMD:C_0603_1608Metric, F.Cu at (9.24, 20.5)
- added C230: 100nF, Capacitor_SMD:C_0603_1608Metric, F.Cu at (9.24, 26.5)
- added C231: 100nF, Capacitor_SMD:C_0603_1608Metric, F.Cu at (15.2, 26.5)
- added C232: 100nF, Capacitor_SMD:C_0603_1608Metric, F.Cu at (27.2, 26.5)
- added C233: 100nF, Capacitor_SMD:C_0603_1608Metric, F.Cu at (33.2, 26.5)
- added C234: 100nF, Capacitor_SMD:C_0603_1608Metric, F.Cu at (45.2, 26.5)
- added C235: 100nF, Capacitor_SMD:C_0603_1608Metric, F.Cu at (51.2, 26.5)
- added C236: 100nF, Capacitor_SMD:C_0603_1608Metric, F.Cu at (63.2, 26.5)
- added C237: 100nF, Capacitor_SMD:C_0603_1608Metric, F.Cu at (69.2, 26.5)
- added C238: 100nF, Capacitor_SMD:C_0603_1608Metric, F.Cu at (87.2, 26.5)
- added C239: 100nF, Capacitor_SMD:C_0603_1608Metric, F.Cu at (93.2, 26.5)
- added C240: 100nF, Capacitor_SMD:C_0603_1608Metric, F.Cu at (99.2, 26.5)
- added C241: 100nF, Capacitor_SMD:C_0603_1608Metric, F.Cu at (105.2, 26.5)
- added C242: 100nF, Capacitor_SMD:C_0603_1608Metric, F.Cu at (111.2, 26.5)
- added C243: 100nF, Capacitor_SMD:C_0603_1608Metric, F.Cu at (123.2, 26.5)
- added C244: 100nF, Capacitor_SMD:C_0603_1608Metric, F.Cu at (129.2, 26.5)
- added C245: 100nF, Capacitor_SMD:C_0603_1608Metric, F.Cu at (135.2, 26.5)
- added C246: 100nF, Capacitor_SMD:C_0603_1608Metric, F.Cu at (147.2, 26.5)
- added C247: 100nF, Capacitor_SMD:C_0603_1608Metric, F.Cu at (153.2, 26.5)
- added C248: 100nF, Capacitor_SMD:C_0603_1608Metric, F.Cu at (159.2, 26.5)
- added C249: 100nF, Capacitor_SMD:C_0603_1608Metric, F.Cu at (165.2, 26.5)
- added C250: 100nF, Capacitor_SMD:C_0603_1608Metric, F.Cu at (171.2, 26.5)
- added C251: 100nF, Capacitor_SMD:C_0603_1608Metric, F.Cu at (189.2, 26.5)
- added C252: 100nF, Capacitor_SMD:C_0603_1608Metric, F.Cu at (195.2, 26.5)
- added C253: 100nF, Capacitor_SMD:C_0603_1608Metric, F.Cu at (207.2, 26.5)
- added C254: 100nF, Capacitor_SMD:C_0603_1608Metric, F.Cu at (213.2, 26.5)
- added C255: 100nF, Capacitor_SMD:C_0603_1608Metric, F.Cu at (225.2, 26.5)
- added C256: 100nF, Capacitor_SMD:C_0603_1608Metric, F.Cu at (231.2, 26.5)
- added C257: 100nF, Capacitor_SMD:C_0603_1608Metric, F.Cu at (243.2, 26.5)
- added C258: 100nF, Capacitor_SMD:C_0603_1608Metric, F.Cu at (249.2, 26.5)
- added C259: 100nF, Capacitor_SMD:C_0603_1608Metric, F.Cu at (249.2, 32.5)
- added C260: 100nF, Capacitor_SMD:C_0603_1608Metric, F.Cu at (243.2, 32.5)
- added C261: 100nF, Capacitor_SMD:C_0603_1608Metric, F.Cu at (231.2, 32.5)
- added C262: 100nF, Capacitor_SMD:C_0603_1608Metric, F.Cu at (225.2, 32.5)
- added C263: 100nF, Capacitor_SMD:C_0603_1608Metric, F.Cu at (213.2, 32.5)
- added C264: 100nF, Capacitor_SMD:C_0603_1608Metric, F.Cu at (207.2, 32.5)
- added C265: 100nF, Capacitor_SMD:C_0603_1608Metric, F.Cu at (201.2, 32.5)
- added C266: 100nF, Capacitor_SMD:C_0603_1608Metric, F.Cu at (195.2, 32.5)
- added C267: 100nF, Capacitor_SMD:C_0603_1608Metric, F.Cu at (189.2, 32.5)
- added C268: 100nF, Capacitor_SMD:C_0603_1608Metric, F.Cu at (183.2, 32.5)
- added C269: 100nF, Capacitor_SMD:C_0603_1608Metric, F.Cu at (177.2, 32.5)
- added C270: 100nF, Capacitor_SMD:C_0603_1608Metric, F.Cu at (171.2, 32.5)
- added C271: 100nF, Capacitor_SMD:C_0603_1608Metric, F.Cu at (159.2, 32.5)
- added C272: 100nF, Capacitor_SMD:C_0603_1608Metric, F.Cu at (153.2, 32.5)
- added C273: 100nF, Capacitor_SMD:C_0603_1608Metric, F.Cu at (147.2, 32.5)
- added C274: 100nF, Capacitor_SMD:C_0603_1608Metric, F.Cu at (141.2, 32.5)
- added C275: 100nF, Capacitor_SMD:C_0603_1608Metric, F.Cu at (135.2, 32.5)
- added C276: 100nF, Capacitor_SMD:C_0603_1608Metric, F.Cu at (129.2, 32.5)
- added C277: 100nF, Capacitor_SMD:C_0603_1608Metric, F.Cu at (123.2, 32.5)
- added C278: 100nF, Capacitor_SMD:C_0603_1608Metric, F.Cu at (117.2, 32.5)
- added C279: 100nF, Capacitor_SMD:C_0603_1608Metric, F.Cu at (111.2, 32.5)
- added C280: 100nF, Capacitor_SMD:C_0603_1608Metric, F.Cu at (105.2, 32.5)
- added C281: 100nF, Capacitor_SMD:C_0603_1608Metric, F.Cu at (87.2, 32.5)
- added C282: 100nF, Capacitor_SMD:C_0603_1608Metric, F.Cu at (81.2, 32.5)
- added C283: 100nF, Capacitor_SMD:C_0603_1608Metric, F.Cu at (75.2, 32.5)
- added C284: 100nF, Capacitor_SMD:C_0603_1608Metric, F.Cu at (69.2, 32.5)
- added C285: 100nF, Capacitor_SMD:C_0603_1608Metric, F.Cu at (63.2, 32.5)
- added C286: 100nF, Capacitor_SMD:C_0603_1608Metric, F.Cu at (57.2, 32.5)
- added C287: 100nF, Capacitor_SMD:C_0603_1608Metric, F.Cu at (51.2, 32.5)
- added C288: 100nF, Capacitor_SMD:C_0603_1608Metric, F.Cu at (45.2, 32.5)
- added C289: 100nF, Capacitor_SMD:C_0603_1608Metric, F.Cu at (33.2, 32.5)
- added C290: 100nF, Capacitor_SMD:C_0603_1608Metric, F.Cu at (27.2, 32.5)
- added C291: 100nF, Capacitor_SMD:C_0603_1608Metric, F.Cu at (15.2, 32.5)
- added C292: 100nF, Capacitor_SMD:C_0603_1608Metric, F.Cu at (9.24, 32.5)
- added C293: 100nF, Capacitor_SMD:C_0603_1608Metric, F.Cu at (9.24, 38.5)
- added C294: 100nF, Capacitor_SMD:C_0603_1608Metric, F.Cu at (15.2, 38.5)
- added C295: 100nF, Capacitor_SMD:C_0603_1608Metric, F.Cu at (21.2, 38.5)
- added C296: 100nF, Capacitor_SMD:C_0603_1608Metric, F.Cu at (27.2, 38.5)
- added C297: 100nF, Capacitor_SMD:C_0603_1608Metric, F.Cu at (33.2, 38.5)
- added C298: 100nF, Capacitor_SMD:C_0603_1608Metric, F.Cu at (39.2, 38.5)
- added C299: 100nF, Capacitor_SMD:C_0603_1608Metric, F.Cu at (45.2, 38.5)
- added C300: 100nF, Capacitor_SMD:C_0603_1608Metric, F.Cu at (51.2, 38.5)
- added C302: 100nF, Capacitor_SMD:C_0603_1608Metric, F.Cu at (69.2, 38.5)
- added C303: 100nF, Capacitor_SMD:C_0603_1608Metric, F.Cu at (81.2, 38.5)
- added C304: 100nF, Capacitor_SMD:C_0603_1608Metric, F.Cu at (87.2, 38.5)
- added C305: 100nF, Capacitor_SMD:C_0603_1608Metric, F.Cu at (93.2, 38.5)
- added C306: 100nF, Capacitor_SMD:C_0603_1608Metric, F.Cu at (99.2, 38.5)
- added C307: 100nF, Capacitor_SMD:C_0603_1608Metric, F.Cu at (105.2, 38.5)
- added C308: 100nF, Capacitor_SMD:C_0603_1608Metric, F.Cu at (117.2, 38.5)
- added C309: 100nF, Capacitor_SMD:C_0603_1608Metric, F.Cu at (123.2, 38.5)
- added C310: 100nF, Capacitor_SMD:C_0603_1608Metric, F.Cu at (129.2, 38.5)
- added C311: 100nF, Capacitor_SMD:C_0603_1608Metric, F.Cu at (135.2, 38.5)
- added C312: 100nF, Capacitor_SMD:C_0603_1608Metric, F.Cu at (141.2, 38.5)
- added C313: 100nF, Capacitor_SMD:C_0603_1608Metric, F.Cu at (153.2, 38.5)
- added C314: 100nF, Capacitor_SMD:C_0603_1608Metric, F.Cu at (159.2, 38.5)
- added C315: 100nF, Capacitor_SMD:C_0603_1608Metric, F.Cu at (165.2, 38.5)
- added C316: 100nF, Capacitor_SMD:C_0603_1608Metric, F.Cu at (171.2, 38.5)
- added C317: 100nF, Capacitor_SMD:C_0603_1608Metric, F.Cu at (177.2, 38.5)
- added C318: 100nF, Capacitor_SMD:C_0603_1608Metric, F.Cu at (189.2, 38.5)
- added C319: 100nF, Capacitor_SMD:C_0603_1608Metric, F.Cu at (195.2, 38.5)
- added C320: 100nF, Capacitor_SMD:C_0603_1608Metric, F.Cu at (207.2, 38.5)
- added C321: 100nF, Capacitor_SMD:C_0603_1608Metric, F.Cu at (213.2, 38.5)
- added C322: 100nF, Capacitor_SMD:C_0603_1608Metric, F.Cu at (219.2, 38.5)
- added C323: 100nF, Capacitor_SMD:C_0603_1608Metric, F.Cu at (225.2, 38.5)
- added C324: 100nF, Capacitor_SMD:C_0603_1608Metric, F.Cu at (231.2, 38.5)
- added C325: 100nF, Capacitor_SMD:C_0603_1608Metric, F.Cu at (237.2, 38.5)
- added C326: 100nF, Capacitor_SMD:C_0603_1608Metric, F.Cu at (243.2, 38.5)
- added C327: 100nF, Capacitor_SMD:C_0603_1608Metric, F.Cu at (249.2, 38.5)
- added C328: 100nF, Capacitor_SMD:C_0603_1608Metric, F.Cu at (249.2, 44.5)
- added C329: 100nF, Capacitor_SMD:C_0603_1608Metric, F.Cu at (231.2, 44.5)
- added C330: 100nF, Capacitor_SMD:C_0603_1608Metric, F.Cu at (225.2, 44.5)
- added C331: 100nF, Capacitor_SMD:C_0603_1608Metric, F.Cu at (213.2, 44.5)
- added C332: 100nF, Capacitor_SMD:C_0603_1608Metric, F.Cu at (207.2, 44.5)
- added C333: 100nF, Capacitor_SMD:C_0603_1608Metric, F.Cu at (195.2, 44.5)
- added C334: 100nF, Capacitor_SMD:C_0603_1608Metric, F.Cu at (189.2, 44.5)
- added C335: 100nF, Capacitor_SMD:C_0603_1608Metric, F.Cu at (177.2, 44.5)
- added C336: 100nF, Capacitor_SMD:C_0603_1608Metric, F.Cu at (171.2, 44.5)
- added C337: 100nF, Capacitor_SMD:C_0603_1608Metric, F.Cu at (159.2, 44.5)
- added C338: 100nF, Capacitor_SMD:C_0603_1608Metric, F.Cu at (153.2, 44.5)
- added C339: 100nF, Capacitor_SMD:C_0603_1608Metric, F.Cu at (141.2, 44.5)
- added C340: 100nF, Capacitor_SMD:C_0603_1608Metric, F.Cu at (135.2, 44.5)
- added C341: 100nF, Capacitor_SMD:C_0603_1608Metric, F.Cu at (129.2, 44.5)
- added C342: 100nF, Capacitor_SMD:C_0603_1608Metric, F.Cu at (123.2, 44.5)
- added C343: 100nF, Capacitor_SMD:C_0603_1608Metric, F.Cu at (117.2, 44.5)
- added C344: 100nF, Capacitor_SMD:C_0603_1608Metric, F.Cu at (105.2, 44.5)
- added C345: 100nF, Capacitor_SMD:C_0603_1608Metric, F.Cu at (99.2, 44.5)
- added C346: 100nF, Capacitor_SMD:C_0603_1608Metric, F.Cu at (87.2, 44.5)
- added C347: 100nF, Capacitor_SMD:C_0603_1608Metric, F.Cu at (81.2, 44.5)
- added C348: 100nF, Capacitor_SMD:C_0603_1608Metric, F.Cu at (69.2, 44.5)
- added C349: 100nF, Capacitor_SMD:C_0603_1608Metric, F.Cu at (63.2, 44.5)
- added C350: 100nF, Capacitor_SMD:C_0603_1608Metric, F.Cu at (51.2, 44.5)
- added C351: 100nF, Capacitor_SMD:C_0603_1608Metric, F.Cu at (45.2, 44.5)
- added C352: 100nF, Capacitor_SMD:C_0603_1608Metric, F.Cu at (33.2, 44.5)
- added C353: 100nF, Capacitor_SMD:C_0603_1608Metric, F.Cu at (27.2, 44.5)
- added C354: 100nF, Capacitor_SMD:C_0603_1608Metric, F.Cu at (9.24, 44.5)
- added C355: 100nF, Capacitor_SMD:C_0603_1608Metric, F.Cu at (9.24, 50.5)
- added C356: 100nF, Capacitor_SMD:C_0603_1608Metric, F.Cu at (15.2, 50.5)
- added C357: 100nF, Capacitor_SMD:C_0603_1608Metric, F.Cu at (21.2, 50.5)
- added C358: 100nF, Capacitor_SMD:C_0603_1608Metric, F.Cu at (27.2, 50.5)
- added C359: 100nF, Capacitor_SMD:C_0603_1608Metric, F.Cu at (33.2, 50.5)
- added C360: 100nF, Capacitor_SMD:C_0603_1608Metric, F.Cu at (39.2, 50.5)
- added C361: 100nF, Capacitor_SMD:C_0603_1608Metric, F.Cu at (45.2, 50.5)
- added C362: 100nF, Capacitor_SMD:C_0603_1608Metric, F.Cu at (51.2, 50.5)
- added C363: 100nF, Capacitor_SMD:C_0603_1608Metric, F.Cu at (57.2, 50.5)
- added C364: 100nF, Capacitor_SMD:C_0603_1608Metric, F.Cu at (63.2, 50.5)
- added C365: 100nF, Capacitor_SMD:C_0603_1608Metric, F.Cu at (69.2, 50.5)
- added C366: 100nF, Capacitor_SMD:C_0603_1608Metric, F.Cu at (75.2, 50.5)
- added C367: 100nF, Capacitor_SMD:C_0603_1608Metric, F.Cu at (81.2, 50.5)
- added C368: 100nF, Capacitor_SMD:C_0603_1608Metric, F.Cu at (87.2, 50.5)
- added C369: 100nF, Capacitor_SMD:C_0603_1608Metric, F.Cu at (99.2, 50.5)
- added C370: 100nF, Capacitor_SMD:C_0603_1608Metric, F.Cu at (105.2, 50.5)
- added C371: 100nF, Capacitor_SMD:C_0603_1608Metric, F.Cu at (111.2, 50.5)
- added C372: 100nF, Capacitor_SMD:C_0603_1608Metric, F.Cu at (117.2, 50.5)
- added C373: 100nF, Capacitor_SMD:C_0603_1608Metric, F.Cu at (123.2, 50.5)
- added C374: 100nF, Capacitor_SMD:C_0603_1608Metric, F.Cu at (129.2, 50.5)
- added C375: 100nF, Capacitor_SMD:C_0603_1608Metric, F.Cu at (135.2, 50.5)
- added C376: 100nF, Capacitor_SMD:C_0603_1608Metric, F.Cu at (141.2, 50.5)
- added C377: 100nF, Capacitor_SMD:C_0603_1608Metric, F.Cu at (147.2, 50.5)
- added C378: 100nF, Capacitor_SMD:C_0603_1608Metric, F.Cu at (153.2, 50.5)
- added C379: 100nF, Capacitor_SMD:C_0603_1608Metric, F.Cu at (159.2, 50.5)
- added C380: 100nF, Capacitor_SMD:C_0603_1608Metric, F.Cu at (171.2, 50.5)
- added C381: 100nF, Capacitor_SMD:C_0603_1608Metric, F.Cu at (177.2, 50.5)
- added C425: 100nF, Capacitor_SMD:C_0603_1608Metric, F.Cu at (183.2, 50.5)
- added C426: 100nF, Capacitor_SMD:C_0603_1608Metric, F.Cu at (189.2, 50.5)
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Connections:
- C4 pad 2: +3.3V -> Net-(RP2350-VREG_AVDD)
- LED117 pad 3: unconnected-(LED117-DOUT-Pad3) -> Net-(LED117-DOUT)
- LED23 pad 1: Net-(LED23-DIN) -> Net-(LED142-DOUT)
- LED28 pad 3: Net-(LED23-DIN) -> Net-(LED123-DIN)
- LED45 pad 3: Net-(LED45-DOUT) -> Net-(LED147-DIN)
- LED50 pad 1: Net-(LED45-DOUT) -> Net-(LED166-DOUT)
- LED60 pad 1: Net-(LED54-DOUT) -> Net-(LED60-DIN)
- LED69 pad 3: Net-(LED69-DOUT) -> Net-(LED171-DIN)
- LED71 pad 3: Net-(LED54-DIN) -> Net-(LED60-DIN)
- LED74 pad 1: Net-(LED69-DOUT) -> Net-(LED190-DOUT)
- LED92 pad 1: Net-(LED86-DOUT) -> Net-(LED80-DOUT)
- LED93 pad 3: Net-(LED93-DOUT) -> Net-(LED195-DIN)
- LED98 pad 1: Net-(LED93-DOUT) -> Net-(LED214-DOUT)
- R10 pad 1: Net-(LED122-DIN) -> unconnected-(R10-Pad1)
- R6 pad 1: +3.3V -> Net-(RP2350-VREG_AVDD)
- RP2350 pad 10: Net-(J2-Pin_5) -> Mute
- RP2350 pad 12: Net-(J2-Pin_4) -> SW8
- RP2350 pad 13: Net-(J2-Pin_3) -> SW7
- RP2350 pad 14: Net-(J2-Pin_2) -> SW6
- RP2350 pad 15: Net-(J2-Pin_1) -> SW5
- RP2350 pad 16: Net-(J3-Pin_4) -> SW4
- RP2350 pad 17: Net-(J3-Pin_3) -> SW3
- RP2350 pad 18: Net-(J3-Pin_2) -> SW2
- RP2350 pad 19: Net-(J3-Pin_1) -> SW1
- RP2350 pad 27: LED_DATA -> unconnected-(RP2350-GPIO16-Pad27)
- RP2350 pad 28: TP_DR -> LED_DATA
- RP2350 pad 46: +3.3V -> Net-(RP2350-VREG_AVDD)
- RP2350 pad 7: ENC_A -> I2S_DIN
- RP2350 pad 8: ENC_B -> I2S_BCLK
- RP2350 pad 9: ENC_SW -> I2S_LRCLK
Routing:
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- added copper zone on B.Cu, net GND
- added copper zone on F.Cu, net GND
Other:
- board size 250.3 x 101.3 mm -> 259 x 101.1 mm
