File: Atrium PCB/Atrium PCB.kicad_pcb (KiCad board)
At the start: 2 copper layers, 259 x 101.1 mm, 995 parts, among them J1 Conn_01x05_Pin, SW2 SKRPACE010, SW3 SKRPACE010, SW41 FG-TC-12E-02-8H, SW49 FG-TC-12E-02-8H, SW55 FG-TC-12E-02-8H, SW56 FG-TC-12E-02-8H, SW57 FG-TC-12E-02-8H, SW58 FG-TC-12E-02-8H, SW59 FG-TC-12E-02-8H, SW60 FG-TC-12E-02-8H, U1 CH604ASR, U10 CH604ASR, U11 CH604ASR, U12 AP2112K-3.3, U13 CH604ASR, U14 CH604ASR, U15 CH604ASR, U16 CH604ASR, U17 CH604ASR, U18 CD74HC4067SM, U19 CH604ASR, U2 LSM6DS3TR-C, U20 CH604ASR, U21 CH604ASR, U22 CH604ASR, U23 CH604ASR, U24 CH604ASR, U25 CH604ASR, U26 CH604ASR, U27 CH604ASR, U28 CH604ASR, U29 CH604ASR, U3 CD74HC4067SM, U30 CH604ASR, U31 CH604ASR, U32 CH604ASR, U33 CH604ASR, U34 CH604ASR, U35 CH604ASR, U36 CH604ASR, U37 CH604ASR, U38 CH604ASR, U39 CH604ASR, U4 CH604ASR, U40 CH604ASR, U41 CH604ASR, U42 CH604ASR, U43 CD74HC4067SM, U44 CH604ASR, U45 CH604ASR, U46 CH604ASR, U47 CH604ASR, U48 MAX98357A, U5 CH604ASR, U6 SN74LVC1T45DBVR, U7 CH604ASR, U8 CH604ASR, U9 CH604ASR, X1 X322512MSB4SI

Commit message: sync
Parts:
- moved C120 5.94 mm to (237.3, 2.50)
- moved LED139 5.94 mm to (237.3, 4.60)
Routing:
- net GND: track 1242.8 -> 1285.6 mm, vias 929 -> 943
- net +3.3V: track 2059.9 -> 2075.4 mm, vias 115 -> 116
- net +5V_LED: track 7451.7 -> 7439.5 mm
- net Net-(LED133-DOUT): track 14.6 -> 8.62 mm
- net Net-(U3-I3): track 61.6 -> 62.6 mm
