File: Atrium PCB/Atrium PCB.kicad_pcb (KiCad board)
At the start: 2 copper layers, 259 x 101.1 mm, 995 parts, among them J1 Conn_01x05_Pin, SW2 SKRPACE010, SW3 SKRPACE010, SW41 FG-TC-12E-02-8H, SW49 FG-TC-12E-02-8H, SW55 FG-TC-12E-02-8H, SW56 FG-TC-12E-02-8H, SW57 FG-TC-12E-02-8H, SW58 FG-TC-12E-02-8H, SW59 FG-TC-12E-02-8H, SW60 FG-TC-12E-02-8H, U1 CH604ASR, U10 CH604ASR, U11 CH604ASR, U12 AP2112K-3.3, U13 CH604ASR, U14 CH604ASR, U15 CH604ASR, U16 CH604ASR, U17 CH604ASR, U18 CD74HC4067SM, U19 CH604ASR, U2 LSM6DS3TR-C, U20 CH604ASR, U21 CH604ASR, U22 CH604ASR, U23 CH604ASR, U24 CH604ASR, U25 CH604ASR, U26 CH604ASR, U27 CH604ASR, U28 CH604ASR, U29 CH604ASR, U3 CD74HC4067SM, U30 CH604ASR, U31 CH604ASR, U32 CH604ASR, U33 CH604ASR, U34 CH604ASR, U35 CH604ASR, U36 CH604ASR, U37 CH604ASR, U38 CH604ASR, U39 CH604ASR, U4 CH604ASR, U40 CH604ASR, U41 CH604ASR, U42 CH604ASR, U43 CD74HC4067SM, U44 CH604ASR, U45 CH604ASR, U46 CH604ASR, U47 CH604ASR, U48 MAX98357A, U5 CH604ASR, U6 SN74LVC1T45DBVR, U7 CH604ASR, U8 CH604ASR, U9 CH604ASR, X1 X322512MSB4SI

Commit message: sync
Parts:
- added G***: LOGO, LOGO, F.Cu at (269.5, 105.9)
- added G***: LOGO, LOGO, F.Cu at (129.4, 50.0)
- added G***: LOGO, LOGO, B.Cu at (129.2, 50.0)
- added G***: LOGO, LOGO, B.Cu at (136.5, 57.8)
Connections:
- LED128 pad 1: unconnected-(LED128-DIN-Pad1) -> Net-(LED128-DIN)
- LED139 pad 3: unconnected-(LED139-DOUT-Pad3) -> Net-(LED128-DIN)
- LED390 pad 1: unconnected-(LED390-DIN-Pad1) -> Net-(LED390-DIN)
- LED411 pad 3: unconnected-(LED411-DOUT-Pad3) -> Net-(LED390-DIN)
Routing:
- net +5V_LED: track 7439.5 -> 7380.3 mm
- net Net-(LED128-DIN): track 0.00 -> 16.0 mm, vias 0 -> 2
- net Net-(LED390-DIN): track 0.00 -> 15.2 mm, vias 0 -> 2
- net GND: track 1285.6 -> 1275.8 mm
- net +3.3V: track 2075.4 -> 2068.6 mm
- net I2S_LRCLK: track 42.1 -> 40.0 mm
- net MUX_3: track 238.0 -> 237.1 mm
- net RP2350_QSPI_SD0: track 11.9 -> 11.2 mm
- net +5V: track 17.9 -> 17.2 mm
- net LED_DIN_A: track 77.3 -> 76.7 mm
